File: hardware/PCBs/Ragnarok_dev/Ragnarok_dev.sch (KiCad schematic (older format))
At the start: 19 parts, among them J1 USB_B_Micro, U1 BMP388, U2 ublox_SAM-M8Q, U3 FT232RL, U4 STM32F427VITx

Commit message: add spi sheet
Parts:
- added C? (x2): 0.1uF, symbol Device:C_Small
- gave numbers to parts that had none: 10
Connections:
- net labels added: BMP_CSB
Other:
- moved on the sheet: U1
Changed lines of the file:
@@
 $Descr A4 11693 8268
 encoding utf-8
-Sheet 1 2
+Sheet 1 3
 Title "Ragnarok Development Board"
 Date "2019-12-18"
 Rev "v0.1"
 Comp "UAH Space Hardware Club"
-Comment1 "Shelby Tull"
+Comment1 ""
 Comment2 "Brennan Haralson"
 Comment3 "Shelby Westrich"
@@
 F 3 "http://www.st.com/st-web-ui/static/active/en/resource/technical/document/datasheet/DM00071990.pdf" H 6250 3750 50  0001 C CNN
 	1    6250 3750
-	1    0    0    -1
-$EndComp
-$Comp
-L BMP388:BMP388 U1
-U 1 1 5DFB015B
-P 9950 1950
-F 0 "U1" H 9950 2717 50  0000 C CNN
-F 1 "BMP388" H 9950 2626 50  0000 C CNN
-F 2 "BMP-388:PQFN50P200X200X80-10N" H 9950 1950 50  0001 L BNN
-F 3 "BOSCH" H 9950 1950 50  0001 L BNN
-F 4 "1.1" H 9950 1950 50  0001 L BNN "Field4"
-F 5 "IPC 7351B" H 9950 1950 50  0001 L BNN "Field5"
-	1    9950 1950
 	1    0    0    -1
 $EndComp
@@
 	4700 1950 5350 1950
 $Comp
-L Switch:SW_SPDT SW?
+L Switch:SW_SPDT SW1
 U 1 1 5E1F0CEE
 P 4800 2250
-F 0 "SW?" H 4650 2050 50  0000 C CNN
+F 0 "SW1" H 4650 2050 50  0000 C CNN
 F 1 "Programming" H 4500 2150 50  0000 C CNN
 F 2 "" H 4800 2250 50  0001 C CNN
@@
 	5150 2250 5150 1550
 $Comp
-L power:+3.3V #PWR?
+L power:+3.3V #PWR0102
 U 1 1 5E1F6902
 P 4600 2150
-F 0 "#PWR?" H 4600 2000 50  0001 C CNN
+F 0 "#PWR0102" H 4600 2000 50  0001 C CNN
 F 1 "+3.3V" V 4615 2278 50  0000 L CNN
 F 2 "" H 4600 2150 50  0001 C CNN
@@
 $EndComp
 $Comp
-L power:GND #PWR?
+L power:GND #PWR0103
 U 1 1 5E1F6FD3
 P 4600 2350
-F 0 "#PWR?" H 4600 2100 50  0001 C CNN
+F 0 "#PWR0103" H 4600 2100 50  0001 C CNN
 F 1 "GND" V 4605 2222 50  0000 R CNN
 F 2 "" H 4600 2350 50  0001 C CNN
@@
 	3000 4400 3100 4400
 $Comp
-L power:GND #PWR?
+L power:GND #PWR0104
 U 1 1 5E1FEDA3
 P 3100 4500
-F 0 "#PWR?" H 3100 4250 50  0001 C CNN
+F 0 "#PWR0104" H 3100 4250 50  0001 C CNN
 F 1 "GND" H 3105 4327 50  0000 C CNN
 F 2 "" H 3100 4500 50  0001 C CNN
@@
 	2700 1150 4700 1150
 $Comp
-L power:+3.3V #PWR?
+L power:+3.3V #PWR0105
 U 1 1 5E2452C8
 P 2800 1500
-F 0 "#PWR?" H 2800 1350 50  0001 C CNN
+F 0 "#PWR0105" H 2800 1350 50  0001 C CNN
 F 1 "+3.3V" H 2815 1673 50  0000 C CNN
 F 2 "" H 2800 1500 50  0001 C CNN
@@
 $EndComp
 $Comp
-L Device:C_Small C?
+L Device:C_Small C13
 U 1 1 5E246F98
 P 1900 2600
-F 0 "C?" V 2129 2600 50  0000 C CNN
+F 0 "C13" V 2129 2600 50  0000 C CNN
 F 1 "0.1uF" V 2038 2600 50  0000 C CNN
 F 2 "" H 1900 2600 50  0001 C CNN
@@
 NoConn ~ 2100 3700
 $Comp
-L Device:LED_Small D?
+L Device:LED_Small D2
 U 1 1 5E2531AF
 P 3950 3900
-F 0 "D?" V 3904 3832 50  0000 R CNN
+F 0 "D2" V 3904 3832 50  0000 R CNN
 F 1 "RX" V 3995 3832 50  0000 R CNN
 F 2 "" V 3950 3900 50  0001 C CNN
@@
 $EndComp
 $Comp
-L Device:LED_Small D?
+L Device:LED_Small D3
 U 1 1 5E255C02
 P 4200 3900
-F 0 "D?" V 4154 3832 50  0000 R CNN
+F 0 "D3" V 4154 3832 50  0000 R CNN
 F 1 "TX" V 4245 3832 50  0000 R CNN
 F 2 "" V 4200 3900 50  0001 C CNN
@@
 $EndComp
 $Comp
-L Device:R_Small R?
+L Device:R_Small R1
 U 1 1 5E25C4C7
 P 3950 4200
-F 0 "R?" H 4009 4246 50  0000 L CNN
+F 0 "R1" H 4009 4246 50  0000 L CNN
 F 1 "270" H 4009 4155 50  0000 L CNN
 F 2 "" H 3950 4200 50  0001 C CNN
@@
 $EndComp
 $Comp
-L Device:R_Small R?
+L Device:R_Small R2
 U 1 1 5E25CD46
 P 4200 4200
-F 0 "R?" H 4259 4246 50  0000 L CNN
+F 0 "R2" H 4259 4246 50  0000 L CNN
 F 1 "270" H 4259 4155 50  0000 L CNN
 F 2 "" H 4200 4200 50  0001 C CNN
@@
 $EndComp
 $Comp
-L power:+3.3V #PWR?
+L power:+3.3V #PWR0106
 U 1 1 5E25CEB1
 P 3950 4500
-F 0 "#PWR?" H 3950 4350 50  0001 C CNN
+F 0 "#PWR0106" H 3950 4350 50  0001 C CNN
 F 1 "+3.3V" H 3965 4673 50  0000 C CNN
 F 2 "" H 3950 4500 50  0001 C CNN
@@
 	5150 1550 5350 1550
 $Comp
-L Device:C_Small C?
+L Device:C_Small C14
 U 1 1 5E27D2E9
 P 3000 1600
-F 0 "C?" V 3100 1500 50  0000 C CNN
+F 0 "C14" V 3100 1500 50  0000 C CNN
 F 1 "10nF" V 3050 1450 50  0000 C CNN
 F 2 "" H 3000 1600 50  0001 C CNN
@@
 $EndComp
 $Comp
-L Device:Ferrite_Bead_Small FB?
+L Device:Ferrite_Bead_Small FB2
 U 1 1 5E27F10E
 P 2800 1800
-F 0 "FB?" H 2900 1846 50  0000 L CNN
+F 0 "FB2" H 2900 1846 50  0000 L CNN
 F 1 "FB" H 2900 1755 50  0000 L CNN
 F 2 "" V 2730 1800 50  0001 C CNN
@@
 $EndComp
 $Comp
-L Device:C_Small C?
+L Device:C_Small C16
 U 1 1 5E284E6E
 P 3100 2250
-F 0 "C?" V 3200 2150 50  0000 C CNN
+F 0 "C16" V 3200 2150 50  0000 C CNN
 F 1 "10nF" V 3150 2100 50  0000 C CNN
 F 2 "" H 3100 2250 50  0001 C CNN
@@
 $EndComp
 $Comp
-L Device:C_Small C?
+L Device:C_Small C15
 U 1 1 5E286D78
 P 3100 2100
-F 0 "C?" V 3200 2000 50  0000 C CNN
+F 0 "C15" V 3200 2000 50  0000 C CNN
 F 1 "10nF" V 3150 1950 50  0000 C CNN
 F 2 "" H 3100 2100 50  0001 C CNN
@@
 Connection ~ 3450 2100
 $Comp
-L power:GND #PWR?
+L power:GND #PWR0107
 U 1 1 5E293D77
 P 3450 1600
-F 0 "#PWR?" H 3450 1350 50  0001 C CNN
+F 0 "#PWR0107" H 3450 1350 50  0001 C CNN
 F 1 "GND" V 3455 1472 50  0000 R CNN
 F 2 "" H 3450 1600 50  0001 C CNN
@@
 Text Label 3700 2700 0    50   ~ 0
 USB_TX
+Text Label 8050 2300 2    50   ~ 0
+BMP_CSB
+$Comp
+L Device:C_Small C?
+U 1 1 5E1881CB
+P 9950 2500
+F 0 "C?" H 10050 2600 50  0000 C CNN
+F 1 "0.1uF" H 10150 2500 50  0000 C CNN
+F 2 "" H 9950 2500 50  0001 C CNN
+F 3 "~" H 9950 2500 50  0001 C CNN
+	1    9950 2500
+	1    0    0    -1
+$EndComp
+$Comp
+L Device:C_Small C?
+U 1 1 5E19130F
+P 9800 2500
+F 0 "C?" H 9900 2600 50  0000 C CNN
+F 1 "0.1uF" H 10000 2500 50  0000 C CNN
+F 2 "" H 9800 2500 50  0001 C CNN
+F 3 "~" H 9800 2500 50  0001 C CNN
+	1    9800 2500
+	-1   0    0    -1
+$EndComp
+$Comp
+L BMP388:BMP388 U1
+U 1 1 5DFB015B
+P 8550 2500
+F 0 "U1" H 8550 3267 50  0000 C CNN
+F 1 "BMP388" H 8550 3176 50  0000 C CNN
+F 2 "BMP-388:PQFN50P200X200X80-10N" H 8550 2500 50  0001 L BNN
+F 3 "BOSCH" H 8550 2500 50  0001 L BNN
+F 4 "1.1" H 8550 2500 50  0001 L BNN "Field4"
+F 5 "IPC 7351B" H 8550 2500 50  0001 L BNN "Field5"
+	1    8550 2500
+	1    0    0    -1
+$EndComp
+$Sheet
+S 8250 950  1100 550
+U 5E1A0CB7
+F0 "SPI Sensors" 50
+F1 "SPI.sch" 50
+$EndSheet
 $EndSCHEMATC

Commit message: Update
Parts:
- removed U1: BMP388, BMP-388:PQFN50P200X200X80-10N, symbol BMP388:BMP388
- added TP1: TestPoint_Probe, symbol Connector:TestPoint_Probe
- added U1: XBee_SMT, RF_Module:Digi_XBee_SMT, symbol RF_ZigBee:XBee_SMT
- gave numbers to parts that had none: 2
Connections:
- net labels removed: BMP_CSB
Other:
- note added: "GET BETTER SYMBOL\n"
- moved on the sheet: C22, C23, H1, H2, H3, H4
Changed lines of the file:
@@
 $Descr A4 11693 8268
 encoding utf-8
-Sheet 1 3
+Sheet 1 4
 Title "Ragnarok Development Board"
 Date "2019-12-18"
@@
 L RF_GPS:ublox_SAM-M8Q U2
 U 1 1 5DFB6E35
-P 9950 3200
-F 0 "U2" H 9950 2611 50  0000 C CNN
-F 1 "ublox_SAM-M8Q" H 9950 2520 50  0000 C CNN
-F 2 "RF_Module:ublox_SAM-M8Q" H 10500 2750 50  0001 C CNN
-F 3 "https://www.u-blox.com/sites/default/files/SAM-M8Q_DataSheet_%28UBX-16012619%29.pdf" H 9950 3200 50  0001 C CNN
-	1    9950 3200
+P 10400 3450
+F 0 "U2" H 10400 2861 50  0000 C CNN
+F 1 "ublox_SAM-M8Q" H 10400 2770 50  0000 C CNN
+F 2 "RF_Module:ublox_SAM-M8Q" H 10950 3000 50  0001 C CNN
+F 3 "https://www.u-blox.com/sites/default/files/SAM-M8Q_DataSheet_%28UBX-16012619%29.pdf" H 10400 3450 50  0001 C CNN
+	1    10400 3450
 	1    0    0    -1
 $EndComp
@@
 L Mechanical:MountingHole H1
 U 1 1 5E041F41
-P 1300 6650
-F 0 "H1" H 1400 6696 50  0000 L CNN
-F 1 "MountingHole" H 1400 6605 50  0000 L CNN
-F 2 "" H 1300 6650 50  0001 C CNN
-F 3 "~" H 1300 6650 50  0001 C CNN
-	1    1300 6650
+P 650 6850
+F 0 "H1" H 750 6896 50  0000 L CNN
+F 1 "MountingHole" H 750 6805 50  0000 L CNN
+F 2 "" H 650 6850 50  0001 C CNN
+F 3 "~" H 650 6850 50  0001 C CNN
+	1    650  6850
 	1    0    0    -1
 $EndComp
@@
 L Mechanical:MountingHole H2
 U 1 1 5E0423C6
-P 1300 6900
-F 0 "H2" H 1400 6946 50  0000 L CNN
-F 1 "MountingHole" H 1400 6855 50  0000 L CNN
-F 2 "" H 1300 6900 50  0001 C CNN
-F 3 "~" H 1300 6900 50  0001 C CNN
-	1    1300 6900
+P 650 7100
+F 0 "H2" H 750 7146 50  0000 L CNN
+F 1 "MountingHole" H 750 7055 50  0000 L CNN
+F 2 "" H 650 7100 50  0001 C CNN
+F 3 "~" H 650 7100 50  0001 C CNN
+	1    650  7100
 	1    0    0    -1
 $EndComp
@@
 L Mechanical:MountingHole H3
 U 1 1 5E04261F
-P 1300 7150
-F 0 "H3" H 1400 7196 50  0000 L CNN
-F 1 "MountingHole" H 1400 7105 50  0000 L CNN
-F 2 "" H 1300 7150 50  0001 C CNN
-F 3 "~" H 1300 7150 50  0001 C CNN
-	1    1300 7150
+P 650 7350
+F 0 "H3" H 750 7396 50  0000 L CNN
+F 1 "MountingHole" H 750 7305 50  0000 L CNN
+F 2 "" H 650 7350 50  0001 C CNN
+F 3 "~" H 650 7350 50  0001 C CNN
+	1    650  7350
 	1    0    0    -1
 $EndComp
@@
 L Mechanical:MountingHole H4
 U 1 1 5E042AA9
-P 1300 7400
-F 0 "H4" H 1400 7446 50  0000 L CNN
-F 1 "MountingHole" H 1400 7355 50  0000 L CNN
-F 2 "" H 1300 7400 50  0001 C CNN
-F 3 "~" H 1300 7400 50  0001 C CNN
-	1    1300 7400
-	1    0    0    -1
-$EndComp
-$Comp
-L Connector:USB_B_Micro J1
-U 1 1 5E045ACF
-P 1000 1800
-F 0 "J1" H 1057 2267 50  0000 C CNN
-F 1 "USB_B_Micro" H 1057 2176 50  0000 C CNN
-F 2 "" H 1150 1750 50  0001 C CNN
-F 3 "~" H 1150 1750 50  0001 C CNN
-	1    1000 1800
+P 650 7600
+F 0 "H4" H 750 7646 50  0000 L CNN
+F 1 "MountingHole" H 750 7555 50  0000 L CNN
+F 2 "" H 650 7600 50  0001 C CNN
+F 3 "~" H 650 7600 50  0001 C CNN
+	1    650  7600
 	1    0    0    -1
 $EndComp
@@
 Text Label 3700 2700 0    50   ~ 0
 USB_TX
-Text Label 8050 2300 2    50   ~ 0
-BMP_CSB
-$Comp
-L Device:C_Small C?
+$Comp
+L Device:C_Small C23
 U 1 1 5E1881CB
-P 9950 2500
-F 0 "C?" H 10050 2600 50  0000 C CNN
-F 1 "0.1uF" H 10150 2500 50  0000 C CNN
-F 2 "" H 9950 2500 50  0001 C CNN
-F 3 "~" H 9950 2500 50  0001 C CNN
-	1    9950 2500
-	1    0    0    -1
-$EndComp
-$Comp
-L Device:C_Small C?
+P 10400 2750
+F 0 "C23" H 10500 2850 50  0000 C CNN
+F 1 "0.1uF" H 10600 2750 50  0000 C CNN
+F 2 "" H 10400 2750 50  0001 C CNN
+F 3 "~" H 10400 2750 50  0001 C CNN
+	1    10400 2750
+	1    0    0    -1
+$EndComp
+$Comp
+L Device:C_Small C22
 U 1 1 5E19130F
-P 9800 2500
-F 0 "C?" H 9900 2600 50  0000 C CNN
-F 1 "0.1uF" H 10000 2500 50  0000 C CNN
-F 2 "" H 9800 2500 50  0001 C CNN
-F 3 "~" H 9800 2500 50  0001 C CNN
-	1    9800 2500
+P 10250 2750
+F 0 "C22" H 10350 2850 50  0000 C CNN
+F 1 "0.1uF" H 10450 2750 50  0000 C CNN
+F 2 "" H 10250 2750 50  0001 C CNN
+F 3 "~" H 10250 2750 50  0001 C CNN
+	1    10250 2750
 	-1   0    0    -1
-$EndComp
-$Comp
-L BMP388:BMP388 U1
-U 1 1 5DFB015B
-P 8550 2500
-F 0 "U1" H 8550 3267 50  0000 C CNN
-F 1 "BMP388" H 8550 3176 50  0000 C CNN
-F 2 "BMP-388:PQFN50P200X200X80-10N" H 8550 2500 50  0001 L BNN
-F 3 "BOSCH" H 8550 2500 50  0001 L BNN
-F 4 "1.1" H 8550 2500 50  0001 L BNN "Field4"
-F 5 "IPC 7351B" H 8550 2500 50  0001 L BNN "Field5"
-	1    8550 2500
-	1    0    0    -1
 $EndComp
 $Sheet
@@
 F1 "SPI.sch" 50
 $EndSheet
+$Sheet
+S 8250 1850 1050 600
+U 5E201923
+F0 "I2C Sensors" 50
+F1 "i2c_sensors.sch" 50
+$EndSheet
+$Comp
+L power:GND #PWR0113
+U 1 1 5E317D31
+P 1000 2200
+F 0 "#PWR0113" H 1000 1950 50  0001 C CNN
+F 1 "GND" H 1100 2050 50  0000 R CNN
+F 2 "" H 1000 2200 50  0001 C CNN
+F 3 "" H 1000 2200 50  0001 C CNN
+	1    1000 2200
+	1    0    0    -1
+$EndComp
+$Comp
+L Connector:USB_B_Micro J1
+U 1 1 5E045ACF
+P 1000 1800
+F 0 "J1" H 1057 2267 50  0000 C CNN
+F 1 "USB_B_Micro" H 1057 2176 50  0000 C CNN
+F 2 "" H 1150 1750 50  0001 C CNN
+F 3 "~" H 1150 1750 50  0001 C CNN
+	1    1000 1800
+	1    0    0    -1
+$EndComp
+$Comp
+L Connector:TestPoint_Probe TP1
+U 1 1 5E36A119
+P 2900 5300
+F 0 "TP1" H 3053 5401 50  0000 L CNN
+F 1 "TestPoint_Probe" H 3053 5310 50  0000 L CNN
+F 2 "" H 3100 5300 50  0001 C CNN
+F 3 "~" H 3100 5300 50  0001 C CNN
+	1    2900 5300
+	1    0    0    -1
+$EndComp
+$Comp
+L RF_ZigBee:XBee_SMT U1
+U 1 1 5E2813EE
+P 9150 5150
+F 0 "U1" H 9150 6331 50  0000 C CNN
+F 1 "XBee_SMT" H 9150 6240 50  0000 C CNN
+F 2 "RF_Module:Digi_XBee_SMT" H 9990 4090 50  0001 C CNN
+F 3 "http://www.digi.com/resources/documentation/digidocs/pdfs/90002126.pdf" H 9150 4750 50  0001 C CNN
+	1    9150 5150
+	1    0    0    -1
+$EndComp
+Text Notes 10200 6100 0    50   ~ 0
+GET BETTER SYMBOL\n
 $EndSCHEMATC

Commit message: UART
Parts:
- removed C23: 0.1uF, symbol Device:C_Small
- removed U1: XBee_SMT, RF_Module:Digi_XBee_SMT, symbol RF_ZigBee:XBee_SMT
- removed U2: ublox_SAM-M8Q, RF_Module:ublox_SAM-M8Q, symbol RF_GPS:ublox_SAM-M8Q
- added LS1: CSS-95B30-SMT, CUI_CSS-95B30-SMT, symbol CSS-95B30-SMT:CSS-95B30-SMT
- added SW2: SW_Push, symbol Switch:SW_Push
- U3: symbol Interface_USB:FT232RL -> Ragnarok_dev-rescue:FT232RL-Interface_USB
Connections:
- net labels added: ABO_CSB, BMP_CSB, Servo1, Servo2, Servo3, Servo4
- wire segments 79 -> 94
Other:
- note added: "Still Need:\n-Openlog\n-Servos\n-Motor Driver\n-Status LEDs\n-Thermistor\n-Voltage Divider\n-Camera\n-Prove points\n-Backup batteries\n-Hookup GPS (sparkfun breakout)\n-3V3 Level Shifting (FTDI)\n-Finish pin assignments\n-Photoresistor/IRLED"
- note removed: "GET BETTER SYMBOL\n"
- moved on the sheet: TP1
Changed lines of the file:
@@
 $Descr A4 11693 8268
 encoding utf-8
-Sheet 1 4
+Sheet 1 5
 Title "Ragnarok Development Board"
 Date "2019-12-18"
@@
 F 3 "http://www.st.com/st-web-ui/static/active/en/resource/technical/document/datasheet/DM00071990.pdf" H 6250 3750 50  0001 C CNN
 	1    6250 3750
-	1    0    0    -1
-$EndComp
-$Comp
-L RF_GPS:ublox_SAM-M8Q U2
-U 1 1 5DFB6E35
-P 10400 3450
-F 0 "U2" H 10400 2861 50  0000 C CNN
-F 1 "ublox_SAM-M8Q" H 10400 2770 50  0000 C CNN
-F 2 "RF_Module:ublox_SAM-M8Q" H 10950 3000 50  0001 C CNN
-F 3 "https://www.u-blox.com/sites/default/files/SAM-M8Q_DataSheet_%28UBX-16012619%29.pdf" H 10400 3450 50  0001 C CNN
-	1    10400 3450
 	1    0    0    -1
 $EndComp
@@
 	6650 850  6650 1050
 Wire Wire Line
-	4800 1050 4800 1750
-Wire Wire Line
 	4800 1750 5350 1750
 Wire Wire Line
@@
 $EndComp
 $Comp
-L Interface_USB:FT232RL U3
+L Ragnarok_dev-rescue:FT232RL-Interface_USB U3
 U 1 1 5DFAFF77
 P 2900 3300
@@
 Text Label 3700 2700 0    50   ~ 0
 USB_TX
-$Comp
-L Device:C_Small C23
-U 1 1 5E1881CB
-P 10400 2750
-F 0 "C23" H 10500 2850 50  0000 C CNN
-F 1 "0.1uF" H 10600 2750 50  0000 C CNN
-F 2 "" H 10400 2750 50  0001 C CNN
-F 3 "~" H 10400 2750 50  0001 C CNN
-	1    10400 2750
-	1    0    0    -1
-$EndComp
-$Comp
-L Device:C_Small C22
-U 1 1 5E19130F
-P 10250 2750
-F 0 "C22" H 10350 2850 50  0000 C CNN
-F 1 "0.1uF" H 10450 2750 50  0000 C CNN
-F 2 "" H 10250 2750 50  0001 C CNN
-F 3 "~" H 10250 2750 50  0001 C CNN
-	1    10250 2750
-	-1   0    0    -1
-$EndComp
 $Sheet
 S 8250 950  1100 550
@@
 F0 "SPI Sensors" 50
 F1 "SPI.sch" 50
+F2 "SCLK" I L 8250 1000 50
+F3 "MOSI" I L 8250 1200 50
+F4 "MISO" O L 8250 1100 50
+F5 "CSB0" I L 8250 1350 50
+F6 "CSB1" I L 8250 1450 50
 $EndSheet
 $Sheet
@@
 L Connector:TestPoint_Probe TP1
 U 1 1 5E36A119
-P 2900 5300
-F 0 "TP1" H 3053 5401 50  0000 L CNN
-F 1 "TestPoint_Probe" H 3053 5310 50  0000 L CNN
-F 2 "" H 3100 5300 50  0001 C CNN
-F 3 "~" H 3100 5300 50  0001 C CNN
-	1    2900 5300
-	1    0    0    -1
-$EndComp
-$Comp
-L RF_ZigBee:XBee_SMT U1
-U 1 1 5E2813EE
-P 9150 5150
-F 0 "U1" H 9150 6331 50  0000 C CNN
-F 1 "XBee_SMT" H 9150 6240 50  0000 C CNN
-F 2 "RF_Module:Digi_XBee_SMT" H 9990 4090 50  0001 C CNN
-F 3 "http://www.digi.com/resources/documentation/digidocs/pdfs/90002126.pdf" H 9150 4750 50  0001 C CNN
-	1    9150 5150
-	1    0    0    -1
-$EndComp
-Text Notes 10200 6100 0    50   ~ 0
-GET BETTER SYMBOL\n
+P 600 6650
+F 0 "TP1" H 753 6751 50  0000 L CNN
+F 1 "TestPoint_Probe" H 753 6660 50  0000 L CNN
+F 2 "" H 800 6650 50  0001 C CNN
+F 3 "~" H 800 6650 50  0001 C CNN
+	1    600  6650
+	1    0    0    -1
+$EndComp
+$Comp
+L Device:C_Small C22
+U 1 1 5E2B31D3
+P 4400 1450
+F 0 "C22" H 4550 1350 50  0000 C CNN
+F 1 "0.1uF" H 4600 1450 50  0000 C CNN
+F 2 "" H 4400 1450 50  0001 C CNN
+F 3 "~" H 4400 1450 50  0001 C CNN
+	1    4400 1450
+	1    0    0    -1
+$EndComp
+Wire Wire Line
+	4800 1050 4800 1750
+$Comp
+L Switch:SW_Push SW2
+U 1 1 5E2B9C0C
+P 4200 1550
+F 0 "SW2" V 4150 1800 50  0000 R CNN
+F 1 "SW_Push" V 4250 1950 50  0000 R CNN
+F 2 "" H 4200 1750 50  0001 C CNN
+F 3 "~" H 4200 1750 50  0001 C CNN
+	1    4200 1550
+	0    -1   1    0
+$EndComp
+$Comp
+L power:GND #PWR0123
+U 1 1 5E2BF907
+P 4200 1850
+F 0 "#PWR0123" H 4200 1600 50  0001 C CNN
+F 1 "GND" H 4250 1700 50  0000 R CNN
+F 2 "" H 4200 1850 50  0001 C CNN
+F 3 "" H 4200 1850 50  0001 C CNN
+	1    4200 1850
+	1    0    0    -1
+$EndComp
+Wire Wire Line
+	5350 1350 4400 1350
+Connection ~ 4400 1350
+Wire Wire Line
+	4400 1350 4200 1350
+Wire Wire Line
+	4400 1550 4400 1800
+Wire Wire Line
+	4400 1800 4200 1800
+Wire Wire Line
+	4200 1800 4200 1850
+Wire Wire Line
+	4200 1750 4200 1800
+Connection ~ 4200 1800
+Text Notes 2700 7050 0    50   ~ 0
+Still Need:\n-Openlog\n-Servos\n-Motor Driver\n-Status LEDs\n-Thermistor\n-Voltage Divider\n-Camera\n-Prove points\n-Backup batteries\n-Hookup GPS (sparkfun breakout)\n-3V3 Level Shifting (FTDI)\n-Finish pin assignments\n-Photoresistor/IRLED
+Text Label 7150 3650 0    50   ~ 0
+USB_TX
+Text Label 7150 3750 0    50   ~ 0
+USB_RX
+Text Label 7150 2150 0    50   ~ 0
+Servo1
+Text Label 7150 2250 0    50   ~ 0
+Servo2
+Text Label 7150 2350 0    50   ~ 0
+Servo3
+Text Label 7150 2450 0    50   ~ 0
+Servo4
+Text Label 7150 5150 0    50   ~ 0
+BMP_CSB
+Text Label 7150 5250 0    50   ~ 0
+ABO_CSB
+Wire Wire Line
+	7150 1850 7500 1850
+Wire Wire Line
+	7500 1850 7500 1000
+Wire Wire Line
+	7500 1000 8250 1000
+Wire Wire Line
+	7150 1950 7600 1950
+Wire Wire Line
+	7600 1950 7600 1100
+Wire Wire Line
+	7600 1100 8250 1100
+Wire Wire Line
+	7150 2050 7700 2050
+Wire Wire Line
+	7700 2050 7700 1200
+Wire Wire Line
+	7700 1200 8250 1200
+Text Label 8250 1350 2    50   ~ 0
+BMP_CSB
+Text Label 8250 1450 2    50   ~ 0
+ABO_CSB
+$Sheet
+S 9550 1600 1350 1000
+U 5E2F29D1
+F0 "UART" 50
+F1 "UART.sch" 50
+F2 "SPS_TX" I L 9550 1700 50
+F3 "SPS_RX" O L 9550 1800 50
+F4 "XB_TX" I L 9550 2000 50
+F5 "XB_RX" O L 9550 2100 50
+F6 "GPS_TX" I L 9550 2300 50
+F7 "GPS_RX" O L 9550 2400 50
+$EndSheet
+$Comp
+L CSS-95B30-SMT:CSS-95B30-SMT LS1
+U 1 1 5E3AF99A
+P 9050 4950
+F 0 "LS1" H 9154 4996 50  0000 L CNN
+F 1 "CSS-95B30-SMT" H 9154 4905 50  0000 L CNN
+F 2 "CUI_CSS-95B30-SMT" H 9050 4950 50  0001 L BNN
+F 3 "CSS-95B30-SMT-TR" H 9050 4950 50  0001 L BNN
+F 4 "CUI" H 9050 4950 50  0001 L BNN "Field4"
+F 5 "Unavailable" H 9050 4950 50  0001 L BNN "Field5"
+F 6 "Audio Buzzer Magnetic 4Vo-p 7Vo-p 80mA 5Vo-p 92dBA Solder Pad Surface Mount T/R" H 9050 4950 50  0001 L BNN "Field6"
+F 7 "CUI Inc." H 9050 4950 50  0001 L BNN "Field7"
+F 8 "None" H 9050 4950 50  0001 L BNN "Field8"
+F 9 "https://www.cui.com/product/audio/buzzers/audio-transducers/magnetic/css-95b30-smt?utm_source=snapeda.com&utm_medium=referral&utm_campaign=snapedaBOM" H 9050 4950 50  0001 L BNN "Field9"
+	1    9050 4950
+	1    0    0    -1
+$EndComp
 $EndSCHEMATC

Commit message: update
Parts:
- added J? (x2): Conn_01x10_Female, symbol Connector:Conn_01x10_Female
- added R?: 31.6k, symbol Device:R_Small
- added R?: 12k, symbol Device:R_Small
- added R?: 10k, symbol Device:R_Small
- added TH?: 10k@25, symbol Device:Thermistor
- added TP2, TP3, TP4, TP5, TP6, TP7: TestPoint_Probe, symbol Connector:TestPoint_Probe
- LS1: value CSS-95B30-SMT -> Buzzer
Connections:
- net +3V3: now also TH?.1
- net GND: now also R?.2, R?.2
- net UART/XB_RX: now also U4.79 (PC11)
- net UART/XB_TX: now also U4.78 (PC10)
- net voltage_div: now reaches U4.24 (PA1)
- net voltage_div: now also R?.1, R?.2
- net voltage_therm: now reaches U4.25 (PA2)
- net voltage_therm: now also R?.1, TH?.2
- net I2C Sensors/SCL: now reaches U4.47 (PB10)
- net I2C Sensors/SDA: now reaches U4.48 (PB11)
- net Servo5: now reaches U4.64 (PC7)
- net GPS_TX: now reaches U4.86 (PD5)
- net GPS_RX: now reaches U4.87 (PD6)
- new net +6V: R?.1
Other:
- note added: "Still Need:\n-Openlog\n-Servos\n-Motor Driver\n-Status LEDs\n-Thermistor\n-Voltage Divider\n-Camera\n-Probe points\n-Backup batteries\n-Hookup GPS (sparkfun breakout)\n-3V3 Level Shifting (FTDI)\n-Finish pin assignments\n-Photoresistor/IRLED"
- note removed: "Still Need:\n-Openlog\n-Servos\n-Motor Driver\n-Status LEDs\n-Thermistor\n-Voltage Divider\n-Camera\n-Prove points\n-Backup batteries\n-Hookup GPS (sparkfun breakout)\n-3V3 Level Shifting (FTDI)\n-Finish pin assignments\n-Photoresistor/IRLED"
- moved on the sheet: LS1
