File: hardware/PCBs/Ragnarok_dev/Ragnarok_dev.sch (KiCad schematic (older format))
At the start: 33 parts, among them J1 USB_B_Micro, SW1 Programming, SW2 SW_Push, U3 FT232RL, U4 STM32F427VITx

Commit message: much schematic work
Parts:
- removed J? (x2): Conn_01x10_Female, symbol Connector:Conn_01x10_Female
- removed LS1: Buzzer, CUI_CSS-95B30-SMT, symbol CSS-95B30-SMT:CSS-95B30-SMT
- added D?: IR, symbol Device:LED_Small
- added D?: 3V3, symbol Device:LED_Small
- added D?: 5V, symbol Device:LED_Small
- added D?: 6V, symbol Device:LED_Small
- added D?: status, symbol Device:LED_Small
- added J?: MAIN_CONN, symbol Connector:Conn_01x14_Female
- added J?: BREAK_CONN, symbol Connector:Conn_01x14_Female
- added J?: JTAG, symbol Connector_Generic:Conn_02x10_Odd_Even
- added LS?: Buzzer, CUI_CMT-8540S-SMT, symbol CMT-8540S-SMT:CMT-8540S-SMT
- added M?: Motor_DC, symbol Motor:Motor_DC
- added Q?: NFET, symbol Device:Q_NMOS_GSD
- added R?: 4.7k, symbol Device:R_Small
- added R? (x4): 300, symbol Device:R_Small
- added R?: 400, symbol Device:R_Small
- added R? (x4): 10k, symbol Device:R_Small
Connections:
- net +3V3: now also D?.2 (A), J?.1 (Pin_1), J?.2 (Pin_2)
- net +6V: now also D?.2 (A), J?.1 (Pin_1), J?.2 (Pin_2)
- net GND: now also J?.10 (Pin_10), J?.12 (Pin_12), J?.12 (Pin_12), J?.13 (Pin_13), J?.14 (Pin_14), J?.14 (Pin_14), J?.16 (Pin_16), J?.18 (Pin_18), J?.20 (Pin_20), J?.4 (Pin_4), J?.6 (Pin_6), J?.8 (Pin_8), Q?.2 (S), R?.2, R?.2, R?.2, R?.2, R?.2, R?.2, R?.2, R?.2, R?.2
- net Servo1: now also J?.4 (Pin_4)
- net Servo2: now also J?.5 (Pin_5)
- net Servo3: now also J?.6 (Pin_6)
- net Servo4: now also J?.7 (Pin_7)
- net Servo5: now also J?.8 (Pin_8)
- net IR_TRANSMIT: now reaches U4.37 (PB2)
- net IR_TRANSMIT: now also D?.2 (A)
- net status_led: now reaches U4.7 (PC13)
- net status_led: now also D?.2 (A)
- net Cam: now reaches U4.71 (PA12)
- net Cam: now also J?.11 (Pin_11)
- net UART/LOG_TX: now reaches U4.80 (PC12)
- net LOG_RX: now reaches U4.83 (PD2)
- net at U4.94 (BOOT0): now also R?.2; no longer SW1.2 (B)
- net speaker_driver: now reaches U4.95 (PB8)
- net speaker_driver: now also Q?.1 (G), R?.1
- net SPS_RX: now reaches U4.97 (PE0)
- net SPS_TX: now reaches U4.98 (PE1)
- new net: R?.1, SW1.2 (B)
- new net: LS?.N, Q?.3 (D)
- new net: D?.1 (K), R?.1 (x5)
- new net: J?.11 (Pin_11), R?.1
- new net: J?.17 (Pin_17), R?.1
- new net: J?.19 (Pin_19), R?.1
- new net +5V: D?.2 (A), J?.3 (Pin_3), LS?.P
- new net Breakout/+5: J?.3 (Pin_3)
- new net Breakout/+6: J?.1 (Pin_1), J?.2 (Pin_2)
- new net Breakout/Cam: J?.11 (Pin_11)
- new net Breakout/GND: J?.12 (Pin_12), J?.13 (Pin_13), J?.14 (Pin_14)
- new net Breakout/Servo1: J?.4 (Pin_4)
- new net Breakout/Servo2: J?.5 (Pin_5)
- new net Breakout/Servo3: J?.6 (Pin_6)
- new net Breakout/Servo4: J?.7 (Pin_7)
- new net Breakout/Servo5: J?.8 (Pin_8)
Other:
- note added: "Fill in"
- note added: "Make sure these line up properly on board"
- note added: "Size: 75(W)x60(L)"
- note added: "Still Need:\n-SPS\n-Motor Driver\n-Camera\n-Probe points\n-Backup batteries\n-3V3 Level Shifting (FTDI)\n-Finish pin assignments"
- note added: "check for better button symbol"
- note added: "just in case"
- note removed: "Still Need:\n-Openlog\n-Servos\n-Motor Driver\n-Status LEDs\n-Thermistor\n-Voltage Divider\n-Camera\n-Probe points\n-Backup batteries\n-Hookup GPS (sparkfun breakout)\n-3V3 Level Shifting (FTDI)\n-Finish pin assignments\n-Photoresistor/IRLED"
- moved on the sheet: H1, H2, H3, H4, R?, SW1, TH?, TP1, TP2, TP3, TP4, TP5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

Commit message: todos
Parts:
- added D?: D_Small, symbol Device:D_Small
- added Q?: NFET, symbol Device:Q_NMOS_GSD
Connections:
- net +6V: now also D?.2 (A)
- net GND: now also M?.2 (-)
- net at M?.1 (+): now also Q?.2 (S)
- new net: D?.1 (K), Q?.3 (D)
- new net motor_driver: Q?.1 (G)
Other:
- note added: "Still Need:\n-SPS\n-Motor Driver\n-Camera\n-Probe points\n-Backup batteries\n-3V3 Level Shifting (FTDI)\n-Fix jumper\n-JTAG\n-Check power supply (source/currents)"
- note added: "needs_assigment"
- note removed: "Still Need:\n-SPS\n-Motor Driver\n-Camera\n-Probe points\n-Backup batteries\n-3V3 Level Shifting (FTDI)\n-Finish pin assignments"
Changed lines of the file:
@@
 Connection ~ 4200 1800
 Text Notes 1950 9450 0    50   ~ 0
-Still Need:\n-SPS\n-Motor Driver\n-Camera\n-Probe points\n-Backup batteries\n-3V3 Level Shifting (FTDI)\n-Finish pin assignments
+Still Need:\n-SPS\n-Motor Driver\n-Camera\n-Probe points\n-Backup batteries\n-3V3 Level Shifting (FTDI)\n-Fix jumper\n-JTAG\n-Check power supply (source/currents)
 Text Label 7150 3650 0    50   ~ 0
 USB_TX
@@
 F3 "+5" I L 9250 2550 50
 F4 "GND" O L 9250 3550 50
-F7 "Servo1" I L 9250 2700 50
-F8 "Servo2" I L 9250 2800 50
-F9 "Servo3" I L 9250 2900 50
-F10 "Servo4" I L 9250 3000 50
-F11 "Servo5" I L 9250 3100 50
-F12 "Cam" I L 9250 3400 50
+F5 "Servo1" I L 9250 2700 50
+F6 "Servo2" I L 9250 2800 50
+F7 "Servo3" I L 9250 2900 50
+F8 "Servo4" I L 9250 3000 50
+F9 "Servo5" I L 9250 3100 50
+F10 "Cam" I L 9250 3400 50
 $EndSheet
 Wire Wire Line
@@
 	1    0    0    -1
 $EndComp
+$Comp
+L Device:Q_NMOS_GSD Q?
+U 1 1 5E5EED42
+P 4300 5450
+F 0 "Q?" H 4505 5496 50  0000 L CNN
+F 1 "NFET" H 4505 5405 50  0000 L CNN
+F 2 "" H 4500 5550 50  0001 C CNN
+F 3 "~" H 4300 5450 50  0001 C CNN
+	1    4300 5450
+	-1   0    0    -1
+$EndComp
+Text Label 4500 5450 0    50   ~ 0
+motor_driver
+Text Notes 4450 5650 0    50   ~ 0
+needs_assigment
+$Comp
+L power:GND #PWR?
+U 1 1 5E5F21BC
+P 4200 6250
+F 0 "#PWR?" H 4200 6000 50  0001 C CNN
+F 1 "GND" H 4205 6077 50  0000 C CNN
+F 2 "" H 4200 6250 50  0001 C CNN
+F 3 "" H 4200 6250 50  0001 C CNN
+	1    4200 6250
+	-1   0    0    -1
+$EndComp
+Wire Wire Line
+	4200 6150 4200 6250
+$Comp
+L power:+6V #PWR?
+U 1 1 5E5FF7E9
+P 4200 4850
+F 0 "#PWR?" H 4200 4700 50  0001 C CNN
+F 1 "+6V" H 4215 5023 50  0000 C CNN
+F 2 "" H 4200 4850 50  0001 C CNN
+F 3 "" H 4200 4850 50  0001 C CNN
+	1    4200 4850
+	1    0    0    -1
+$EndComp
+$Comp
+L Device:D_Small D?
+U 1 1 5E608838
+P 4200 5050
+F 0 "D?" V 4246 4982 50  0000 R CNN
+F 1 "D_Small" V 4155 4982 50  0000 R CNN
+F 2 "" V 4200 5050 50  0001 C CNN
+F 3 "~" V 4200 5050 50  0001 C CNN
+	1    4200 5050
+	0    -1   -1   0
+$EndComp
+Wire Wire Line
+	4200 4850 4200 4950
+Wire Wire Line
+	4200 5150 4200 5250
 $EndSCHEMATC

Commit message: update
Parts:
- removed J?: MAIN_CONN, symbol Connector:Conn_01x14_Female
- removed J?: BREAK_CONN, symbol Connector:Conn_01x14_Female
- removed TP3, TP4, TP5, TP6, TP7: TestPoint_Probe, symbol Connector:TestPoint_Probe
- added J2: BOARD_CONN, symbol Connector:Conn_01x12_Female
- added J3: BREAK_CONN, symbol Connector:Conn_01x12_Female
- C13, C14, C15, C16, C22: footprint (none) -> Capacitor_SMD:C_0603_1608Metric_Pad1.05x0.95mm_HandSolder
- D1, D4, D5, D6: renamed from D?; footprint (none) -> LED_SMD:LED_0603_1608Metric_Pad1.05x0.95mm_HandSolder
- D2, D3: footprint (none) -> LED_SMD:LED_0603_1608Metric_Pad1.05x0.95mm_HandSolder
- D7: renamed from D?; footprint (none) -> Connector_JST:JST_GH_SM02B-GHS-TB_1x02-1MP_P1.25mm_Horizontal
- D8: renamed from D?; footprint (none) -> Diode_SMD:D_0603_1608Metric_Pad1.05x0.95mm_HandSolder
- FB2: footprint (none) -> Inductor_SMD:L_0603_1608Metric_Pad1.05x0.95mm_HandSolder
- H1, H2, H3, H4: footprint (none) -> MountingHole:MountingHole_2.2mm_M2
- LS1: renamed from LS?; footprint CUI_CMT-8540S-SMT -> cmt-buzzer:CUI_CMT-8540S-SMT
- M1: renamed from M?; footprint (none) -> Connector_JST:JST_GH_SM02B-GHS-TB_1x02-1MP_P1.25mm_Horizontal
- R1, R2: footprint (none) -> Resistor_SMD:R_0603_1608Metric_Pad1.05x0.95mm_HandSolder
- R10, R11, R12, R13, R14, R15, R16, R17, R18, R6, R7, R8, R9: renamed from R?; footprint (none) -> Resistor_SMD:R_0603_1608Metric_Pad1.05x0.95mm_HandSolder
- TH1: renamed from TH?; footprint (none) -> Connector_JST:JST_GH_SM02B-GHS-TB_1x02-1MP_P1.25mm_Horizontal
- TP1: value TestPoint_Probe -> TP_USBTX; footprint (none) -> TestPoint:TestPoint_Pad_1.0x1.0mm
- TP2: value TestPoint_Probe -> TP_USBRX; footprint (none) -> TestPoint:TestPoint_Pad_1.0x1.0mm
- gave numbers to parts that had none: 3
Connections:
- net +5V: now also J2.3 (Pin_3)
- net +6V: now also J2.1 (Pin_1), J2.2 (Pin_2)
- net Breakout/+5: now also J3.3 (Pin_3)
- net Breakout/+6: now also J3.1 (Pin_1), J3.2 (Pin_2)
- net Breakout/Cam: now also J3.9 (Pin_9)
- net Breakout/GND: now also J3.10 (Pin_10), J3.11 (Pin_11), J3.12 (Pin_12)
- net Breakout/Servo1: now also J3.4 (Pin_4)
- net Breakout/Servo2: now also J3.5 (Pin_5)
- net Breakout/Servo3: now also J3.6 (Pin_6)
- net Breakout/Servo4: now also J3.7 (Pin_7)
- net Breakout/Servo5: now also J3.8 (Pin_8)
- net Cam: now also J2.9 (Pin_9)
- net GND: now also J2.10 (Pin_10), J2.11 (Pin_11), J2.12 (Pin_12)
- net Servo1: now also J2.4 (Pin_4)
- net Servo2: now also J2.5 (Pin_5)
- net Servo3: now also J2.6 (Pin_6)
- net Servo4: now also J2.7 (Pin_7)
- net Servo5: now also J2.8 (Pin_8)
- net USB_RX: now also TP2.1
- net USB_TX: now also TP1.1
- net motor_driver: now also U4.96 (PB9)
- net TMS: now reaches U4.72 (PA13)
- net TMS: now also J4.7 (Pin_7)
- net TCK: now reaches U4.76 (PA14)
- net TCK: now also J4.9 (Pin_9)
- net JTDI: now reaches U4.77 (PA15)
- net JTDI: now also J4.5 (Pin_5)
- net JTDO: now reaches U4.89 (PB3)
- net JTDO: now also J4.13 (Pin_13)
- net nTRST: now reaches U4.90 (PB4)
- net nTRST: now also J4.3 (Pin_3)
- net nSRST: now reaches J4.15 (Pin_15)
Other:
- note removed: "Fill in"
- note removed: "Still Need:\n-SPS\n-Motor Driver\n-Camera\n-Probe points\n-Backup batteries\n-3V3 Level Shifting (FTDI)\n-Fix jumper\n-JTAG\n-Check power supply (source/currents)"
- note removed: "needs_assigment"
- moved on the sheet: TP2

Commit message: finish schematic
Parts:
- J1: footprint (none) -> Connector_USB:USB_Micro-B_Amphenol_10103594-0001LF_Horizontal
- J2: footprint (none) -> Connector_PinHeader_1.27mm:PinHeader_1x12_P1.27mm_Vertical_SMD_Pin1Left
- J3: footprint (none) -> Connector_PinHeader_1.27mm:PinHeader_1x12_P1.27mm_Vertical_SMD_Pin1Right
- J4: footprint (none) -> Connector_PinSocket_2.00mm:PinSocket_2x10_P2.00mm_Vertical
- Q1, Q2: footprint (none) -> Package_TO_SOT_SMD:SOT-23_Handsoldering
- SW1: footprint (none) -> CS12 Switch:CS12ANW03
- SW2: footprint (none) -> Button_Switch_SMD:SW_SPST_B3SL-1022P
Changed lines of the file:
@@
 F 0 "SW1" H 4350 2050 50  0000 C CNN
 F 1 "Programming" H 4200 2150 50  0000 C CNN
-F 2 "" H 4500 2250 50  0001 C CNN
+F 2 "CS12 Switch:CS12ANW03" H 4500 2250 50  0001 C CNN
 F 3 "" H 4500 2250 50  0001 C CNN
 	1    4500 2250
@@
 F 0 "J1" H 1057 2267 50  0000 C CNN
 F 1 "USB_B_Micro" H 1057 2176 50  0000 C CNN
-F 2 "" H 1150 1750 50  0001 C CNN
+F 2 "Connector_USB:USB_Micro-B_Amphenol_10103594-0001LF_Horizontal" H 1150 1750 50  0001 C CNN
 F 3 "~" H 1150 1750 50  0001 C CNN
 	1    1000 1800
@@
 F 0 "SW2" V 4150 1800 50  0000 R CNN
 F 1 "SW_Push" V 4250 1950 50  0000 R CNN
-F 2 "" H 4200 1750 50  0001 C CNN
+F 2 "Button_Switch_SMD:SW_SPST_B3SL-1022P" H 4200 1750 50  0001 C CNN
 F 3 "~" H 4200 1750 50  0001 C CNN
 	1    4200 1550
@@
 F 0 "Q1" H 2905 7046 50  0000 L CNN
 F 1 "NFET" H 2905 6955 50  0000 L CNN
-F 2 "" H 2900 7100 50  0001 C CNN
+F 2 "Package_TO_SOT_SMD:SOT-23_Handsoldering" H 2900 7100 50  0001 C CNN
 F 3 "~" H 2700 7000 50  0001 C CNN
 	1    2700 7000
@@
 F 0 "J4" H 10200 5817 50  0000 C CNN
 F 1 "JTAG" H 10200 5726 50  0000 C CNN
-F 2 "" H 10150 5200 50  0001 C CNN
+F 2 "Connector_PinSocket_2.00mm:PinSocket_2x10_P2.00mm_Vertical" H 10150 5200 50  0001 C CNN
 F 3 "~" H 10150 5200 50  0001 C CNN
 	1    10150 5200
@@
 F 0 "Q2" H 4505 5496 50  0000 L CNN
 F 1 "NFET" H 4505 5405 50  0000 L CNN
-F 2 "" H 4500 5550 50  0001 C CNN
+F 2 "Package_TO_SOT_SMD:SOT-23_Handsoldering" H 4500 5550 50  0001 C CNN
 F 3 "~" H 4300 5450 50  0001 C CNN
 	1    4300 5450
@@
 F 0 "J2" H 8450 2250 50  0000 L CNN
 F 1 "BOARD_CONN" H 8400 2150 50  0000 L CNN
-F 2 "" H 8600 2950 50  0001 C CNN
+F 2 "Connector_PinHeader_1.27mm:PinHeader_1x12_P1.27mm_Vertical_SMD_Pin1Left" H 8600 2950 50  0001 C CNN
 F 3 "~" H 8600 2950 50  0001 C CNN
 	1    8600 2950
@@
 F 0 "J3" H 8700 3700 50  0000 L CNN
 F 1 "BREAK_CONN" H 8400 3600 50  0000 L CNN
-F 2 "" H 8650 2950 50  0001 C CNN
+F 2 "Connector_PinHeader_1.27mm:PinHeader_1x12_P1.27mm_Vertical_SMD_Pin1Right" H 8650 2950 50  0001 C CNN
 F 3 "~" H 8650 2950 50  0001 C CNN
 	1    8650 2950
