File: hardware/PCBs/Ragnarok_dev/Ragnarok_dev.sch (KiCad schematic (older format))
At the start: 48 parts, among them J1 USB_B_Micro, J2 BOARD_CONN, J3 BREAK_CONN, J4 JTAG, M1 Motor_DC, Q1 NFET, Q2 NFET, SW1 Programming, SW2 SW_Push, U3 FT232RL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

Commit message: begin layout
Parts:
- added H5, H6, H7, H8: MountingHole, MountingHole:MountingHole_2.2mm_M2, symbol Mechanical:MountingHole
- J2: footprint Connector_PinHeader_1.27mm:PinHeader_1x12_P1.27mm_Vertical_SMD_Pin1Left -> Connector_PinHeader_1.27mm:PinHeader_1x12_P1.27mm_Vertical
- J3: footprint Connector_PinHeader_1.27mm:PinHeader_1x12_P1.27mm_Vertical_SMD_Pin1Right -> Connector_PinHeader_1.27mm:PinHeader_1x12_P1.27mm_Vertical
Changed lines of the file:
@@
 F 0 "J2" H 8450 2250 50  0000 L CNN
 F 1 "BOARD_CONN" H 8400 2150 50  0000 L CNN
-F 2 "Connector_PinHeader_1.27mm:PinHeader_1x12_P1.27mm_Vertical_SMD_Pin1Left" H 8600 2950 50  0001 C CNN
+F 2 "Connector_PinHeader_1.27mm:PinHeader_1x12_P1.27mm_Vertical" H 8600 2950 50  0001 C CNN
 F 3 "~" H 8600 2950 50  0001 C CNN
 	1    8600 2950
@@
 F 0 "J3" H 8700 3700 50  0000 L CNN
 F 1 "BREAK_CONN" H 8400 3600 50  0000 L CNN
-F 2 "Connector_PinHeader_1.27mm:PinHeader_1x12_P1.27mm_Vertical_SMD_Pin1Right" H 8650 2950 50  0001 C CNN
+F 2 "Connector_PinHeader_1.27mm:PinHeader_1x12_P1.27mm_Vertical" H 8650 2950 50  0001 C CNN
 F 3 "~" H 8650 2950 50  0001 C CNN
 	1    8650 2950
@@
 Wire Wire Line
 	4000 2800 4100 2800
+$Comp
+L Mechanical:MountingHole H5
+U 1 1 5E8F0613
+P 650 5400
+F 0 "H5" H 750 5446 50  0000 L CNN
+F 1 "MountingHole" H 750 5355 50  0000 L CNN
+F 2 "MountingHole:MountingHole_2.2mm_M2" H 650 5400 50  0001 C CNN
+F 3 "~" H 650 5400 50  0001 C CNN
+	1    650  5400
+	1    0    0    -1
+$EndComp
+$Comp
+L Mechanical:MountingHole H6
+U 1 1 5E8F0619
+P 650 5650
+F 0 "H6" H 750 5696 50  0000 L CNN
+F 1 "MountingHole" H 750 5605 50  0000 L CNN
+F 2 "MountingHole:MountingHole_2.2mm_M2" H 650 5650 50  0001 C CNN
+F 3 "~" H 650 5650 50  0001 C CNN
+	1    650  5650
+	1    0    0    -1
+$EndComp
+$Comp
+L Mechanical:MountingHole H7
+U 1 1 5E8F061F
+P 650 5900
+F 0 "H7" H 750 5946 50  0000 L CNN
+F 1 "MountingHole" H 750 5855 50  0000 L CNN
+F 2 "MountingHole:MountingHole_2.2mm_M2" H 650 5900 50  0001 C CNN
+F 3 "~" H 650 5900 50  0001 C CNN
+	1    650  5900
+	1    0    0    -1
+$EndComp
+$Comp
+L Mechanical:MountingHole H8
+U 1 1 5E8F0625
+P 650 6150
+F 0 "H8" H 750 6196 50  0000 L CNN
+F 1 "MountingHole" H 750 6105 50  0000 L CNN
+F 2 "MountingHole:MountingHole_2.2mm_M2" H 650 6150 50  0001 C CNN
+F 3 "~" H 650 6150 50  0001 C CNN
+	1    650  6150
+	1    0    0    -1
+$EndComp
 $EndSCHEMATC

Commit message: first PCB
Parts:
- J2, J3: footprint Connector_PinHeader_1.27mm:PinHeader_1x12_P1.27mm_Vertical -> ragnarok_custom_libs:Board_Jumper
Connections:
- net Breakout/+5: now also J3.10 (Pin_10); no longer J3.3 (Pin_3)
- net Breakout/+6: now also J3.11 (Pin_11), J3.12 (Pin_12); no longer J3.1 (Pin_1), J3.2 (Pin_2)
- net Breakout/Cam: now also J3.4 (Pin_4); no longer J3.9 (Pin_9)
- net Breakout/GND: now also J3.1 (Pin_1), J3.2 (Pin_2), J3.3 (Pin_3); no longer J3.10 (Pin_10), J3.11 (Pin_11), J3.12 (Pin_12)
- net Breakout/Servo1: now also J3.9 (Pin_9); no longer J3.4 (Pin_4)
- net Breakout/Servo2: now also J3.8 (Pin_8); no longer J3.5 (Pin_5)
- net Breakout/Servo3: now also J3.7 (Pin_7); no longer J3.6 (Pin_6)
- net Breakout/Servo4: now also J3.6 (Pin_6); no longer J3.7 (Pin_7)
- net Breakout/Servo5: now also J3.5 (Pin_5); no longer J3.8 (Pin_8)
Changed lines of the file:
@@
 F 0 "J2" H 8450 2250 50  0000 L CNN
 F 1 "BOARD_CONN" H 8400 2150 50  0000 L CNN
-F 2 "Connector_PinHeader_1.27mm:PinHeader_1x12_P1.27mm_Vertical" H 8600 2950 50  0001 C CNN
+F 2 "ragnarok_custom_libs:Board_Jumper" H 8600 2950 50  0001 C CNN
 F 3 "~" H 8600 2950 50  0001 C CNN
 	1    8600 2950
@@
 L Connector:Conn_01x12_Female J3
 U 1 1 5E7127DC
-P 8650 2950
-F 0 "J3" H 8700 3700 50  0000 L CNN
-F 1 "BREAK_CONN" H 8400 3600 50  0000 L CNN
-F 2 "Connector_PinHeader_1.27mm:PinHeader_1x12_P1.27mm_Vertical" H 8650 2950 50  0001 C CNN
-F 3 "~" H 8650 2950 50  0001 C CNN
-	1    8650 2950
-	-1   0    0    -1
+P 8650 3050
+F 0 "J3" H 8550 2250 50  0000 L CNN
+F 1 "BREAK_CONN" H 8250 2300 50  0000 L CNN
+F 2 "ragnarok_custom_libs:Board_Jumper" H 8650 3050 50  0001 C CNN
+F 3 "~" H 8650 3050 50  0001 C CNN
+	1    8650 3050
+	-1   0    0    1
 $EndComp
 Text Label 7150 3950 0    50   ~ 0
