File: hardware/PCBs/Ragnarok_dev/power_supply.sch (KiCad schematic (older format))
At the start: 29 parts, among them Q1 Q_PMOS_GDS, Q2 Q_PMOS_GDS, SW3 Power, U5 TPS62142, U6 RT9069-50GB

Commit message: update
Parts:
- removed D1: USB_PROTECTION, symbol Device:D_Small
- removed Q1, Q2: Q_PMOS_GDS, Package_TO_SOT_SMD:SOT-223-3_TabPin2, symbol Device:Q_PMOS_GDS
- added D10, D9: USB_PROTECTION, Diode_SMD:D_0603_1608Metric_Pad1.05x0.95mm_HandSolder, symbol Device:D_Small
- added Q3: Q_NMOS_GDS, symbol Device:Q_NMOS_GDS
- added Q4, Q5: Q_PMOS_GDS, Package_TO_SOT_SMD:SOT-223-3_TabPin2, symbol Device:Q_PMOS_GDS
- added R19, R20, R21: 10k, Resistor_SMD:R_0603_1608Metric_Pad1.05x0.95mm_HandSolder, symbol Device:R_Small
- BT1: footprint (none) -> Connector_JST:JST_GH_SM02B-GHS-TB_1x02-1MP_P1.25mm_Horizontal
- C24, C25: footprint (none) -> Capacitor_SMD:C_0603_1608Metric_Pad1.05x0.95mm_HandSolder
- FB1, L1: footprint (none) -> Inductor_SMD:L_0603_1608Metric_Pad1.05x0.95mm_HandSolder
- R3: footprint (none) -> Resistor_SMD:R_0603_1608Metric_Pad1.05x0.95mm_HandSolder
- U6: footprint (none) -> Package_TO_SOT_SMD:SOT-23-5
Connections:
- net +BATT: now also D10.2 (A), Q3.1 (G), R19.1
- net GND: now also Q3.3 (S), R19.2, R21.2
- net USB_VIN: now also D9.2 (A)
- net at SW3.2 (B): now also D10.1 (K), Q5.3 (S)
- new net: Q4.3 (S), Q5.1 (G), R21.1
- new net: D9.1 (K), Q4.2 (D), Q5.2 (D), R20.1
- new net: Q3.2 (D), Q4.1 (G), R20.2
Other:
- note removed: "Default battery\nUSB power should only be connected if there are no batteries connected"
- note removed: "Disconnects the USB power if a battery is connected"
- note removed: "Prevents against reverse voltage"
- note removed: "Really need to look into the feasibility of this"
- note removed: "This needs to be fixed , currently floats\n"

Commit message: finish schematic
Parts:
- removed Q3: Q_NMOS_GDS, symbol Device:Q_NMOS_GDS
- removed Q4, Q5: Q_PMOS_GDS, Package_TO_SOT_SMD:SOT-223-3_TabPin2, symbol Device:Q_PMOS_GDS
- added Q3: Q_NMOS_GSD, Package_TO_SOT_SMD:SOT-23_Handsoldering, symbol Device:Q_NMOS_GSD
- added Q4, Q5: Q_PMOS_GSD, Package_TO_SOT_SMD:SOT-23_Handsoldering, symbol Device:Q_PMOS_GSD
- SW3: footprint (none) -> CS12 Switch:CS12ANW03
Connections:
- net +BATT: now also Q3.1 (G)
- net GND: now also Q3.2 (S)
- net at R21.1: now also Q4.2 (S), Q5.1 (G)
- net at D9.1 (K), R20.1: now also Q4.3 (D), Q5.3 (D)
- net at D10.1 (K), SW3.2 (B): now also Q5.2 (S)
- net at R20.2: now also Q3.3 (D), Q4.1 (G)
Changed lines of the file:
@@
 Wire Wire Line
 	6850 2600 7100 2600
-$Comp
-L Device:Q_PMOS_GDS Q5
-U 1 1 5E678129
-P 4800 1200
-F 0 "Q5" V 5143 1200 50  0000 C CNN
-F 1 "Q_PMOS_GDS" V 5052 1200 50  0000 C CNN
-F 2 "Package_TO_SOT_SMD:SOT-223-3_TabPin2" H 5000 1300 50  0001 C CNN
-F 3 "~" H 4800 1200 50  0001 C CNN
-	1    4800 1200
-	0    -1   -1   0
-$EndComp
-$Comp
-L Device:Q_NMOS_GDS Q3
-U 1 1 5E679753
-P 4200 2100
-F 0 "Q3" H 4404 2146 50  0000 L CNN
-F 1 "Q_NMOS_GDS" H 4404 2055 50  0000 L CNN
-F 2 "" H 4400 2200 50  0001 C CNN
-F 3 "~" H 4200 2100 50  0001 C CNN
-	1    4200 2100
-	1    0    0    -1
-$EndComp
 Text HLabel 3900 1100 0    50   Input ~ 0
 USB_VIN
@@
 F 0 "SW3" H 6200 900 50  0000 C CNN
 F 1 "Power" H 6150 1000 50  0000 C CNN
-F 2 "" H 6350 1100 50  0001 C CNN
+F 2 "CS12 Switch:CS12ANW03" H 6350 1100 50  0001 C CNN
 F 3 "" H 6350 1100 50  0001 C CNN
 	1    6350 1100
@@
 $EndComp
 NoConn ~ 6550 1000
-$Comp
-L Device:Q_PMOS_GDS Q4
-U 1 1 5E752755
-P 4450 1500
-F 0 "Q4" V 4793 1500 50  0000 C CNN
-F 1 "Q_PMOS_GDS" V 4702 1500 50  0000 C CNN
-F 2 "Package_TO_SOT_SMD:SOT-223-3_TabPin2" H 4650 1600 50  0001 C CNN
-F 3 "~" H 4450 1500 50  0001 C CNN
-	1    4450 1500
-	0    -1   -1   0
-$EndComp
-Wire Wire Line
-	4650 1400 4800 1400
 $Comp
 L Device:R_Small R19
@@
 $EndComp
 Connection ~ 3700 1850
+$Comp
+L Device:Q_NMOS_GSD Q3
+U 1 1 5E6487E5
+P 4200 2100
+F 0 "Q3" H 4406 2146 50  0000 L CNN
+F 1 "Q_NMOS_GSD" H 4406 2055 50  0000 L CNN
+F 2 "Package_TO_SOT_SMD:SOT-23_Handsoldering" H 4400 2200 50  0001 C CNN
+F 3 "~" H 4200 2100 50  0001 C CNN
+	1    4200 2100
+	1    0    0    -1
+$EndComp
+$Comp
+L Device:Q_PMOS_GSD Q4
+U 1 1 5E67580A
+P 4450 1500
+F 0 "Q4" V 4793 1500 50  0000 C CNN
+F 1 "Q_PMOS_GSD" V 4702 1500 50  0000 C CNN
+F 2 "Package_TO_SOT_SMD:SOT-23_Handsoldering" H 4650 1600 50  0001 C CNN
+F 3 "~" H 4450 1500 50  0001 C CNN
+	1    4450 1500
+	0    -1   -1   0
+$EndComp
+$Comp
+L Device:Q_PMOS_GSD Q5
+U 1 1 5E67BC2B
+P 4800 1200
+F 0 "Q5" V 5143 1200 50  0000 C CNN
+F 1 "Q_PMOS_GSD" V 5052 1200 50  0000 C CNN
+F 2 "Package_TO_SOT_SMD:SOT-23_Handsoldering" H 5000 1300 50  0001 C CNN
+F 3 "~" H 4800 1200 50  0001 C CNN
+	1    4800 1200
+	0    -1   -1   0
+$EndComp
+Wire Wire Line
+	4650 1400 4800 1400
 $EndSCHEMATC
