File: hardware/PCBs/Ragnarok_dev/i2c_sensors.sch (KiCad schematic (older format))
At the start: 10 parts, among them J2 SPS30, U10 SDP32, U9 BNO055

Commit message: UART
Parts:
- removed J2: SPS30, symbol Connector:Conn_01x05_Female
- U10: footprint XDCR_SDP32-125PA-TR-250PCS -> SDP32-125PA-TR-250PCS:XDCR_SDP32-125PA-TR-250PCS
Other:
- note removed: "Addr: 0x69\n"
- note removed: "GND"
- note removed: "SCL"
- note removed: "SEL\n"
- note removed: "VDD\n"
Changed lines of the file:
@@
 $Descr A4 11693 8268
 encoding utf-8
-Sheet 4 4
+Sheet 4 5
 Title ""
 Date ""
@@
 $EndComp
 $Comp
-L Connector:Conn_01x05_Female J2
-U 1 1 5E20A41B
-P 4850 7050
-F 0 "J2" H 4750 7500 50  0000 L CNN
-F 1 "SPS30" H 4650 7400 50  0000 L CNN
-F 2 "" H 4850 7050 50  0001 C CNN
-F 3 "~" H 4850 7050 50  0001 C CNN
-	1    4850 7050
-	1    0    0    -1
-$EndComp
-Text Notes 4850 6850 0    50   ~ 0
-VDD\n
-Text Notes 4850 6950 0    50   ~ 0
-SDA
-Text Notes 4850 7050 0    50   ~ 0
-SCL
-Text Notes 4850 7150 0    50   ~ 0
-SEL\n
-Text Notes 4850 7250 0    50   ~ 0
-GND
-$Comp
 L SDP32-125PA-TR-250PCS:SDP32-125PA-TR-250PCS U10
 U 1 1 5E20C00D
@@
 F 0 "U10" H 5250 5967 50  0000 C CNN
 F 1 "SDP32" H 5250 5876 50  0000 C CNN
-F 2 "XDCR_SDP32-125PA-TR-250PCS" H 5250 5300 50  0001 L BNN
+F 2 "SDP32-125PA-TR-250PCS:XDCR_SDP32-125PA-TR-250PCS" H 5250 5300 50  0001 L BNN
 F 3 "4.4mm" H 5250 5300 50  0001 L BNN
 F 4 "SENSIRION" H 5250 5300 50  0001 L BNN "Field4"
@@
 	4250 3050 4250 5400
 Wire Wire Line
-	4250 5400 4250 6950
-Connection ~ 4250 5400
-Wire Wire Line
 	4150 3150 4150 5300
-Connection ~ 4150 5300
-Wire Wire Line
-	4150 5300 4150 7050
 $Comp
 L Device:C_Small C33
@@
 	6100 5700 6000 5700
 Wire Wire Line
-	4250 6950 4650 6950
-Wire Wire Line
-	4150 7050 4650 7050
-Wire Wire Line
-	4650 7150 4550 7150
-Wire Wire Line
-	4550 7150 4550 7250
-Wire Wire Line
-	4550 7250 4650 7250
-$Comp
-L power:GND #PWR0123
-U 1 1 5E338AEB
-P 4550 7350
-F 0 "#PWR0123" H 4550 7100 50  0001 C CNN
-F 1 "GND" H 4555 7177 50  0000 C CNN
-F 2 "" H 4550 7350 50  0001 C CNN
-F 3 "" H 4550 7350 50  0001 C CNN
-	1    4550 7350
-	1    0    0    -1
-$EndComp
-Wire Wire Line
-	4550 7250 4550 7350
-Connection ~ 4550 7250
-$Comp
-L power:+3.3V #PWR0124
-U 1 1 5E33A2C4
-P 4550 6750
-F 0 "#PWR0124" H 4550 6600 50  0001 C CNN
-F 1 "+3.3V" H 4565 6923 50  0000 C CNN
-F 2 "" H 4550 6750 50  0001 C CNN
-F 3 "" H 4550 6750 50  0001 C CNN
-	1    4550 6750
-	1    0    0    -1
-$EndComp
-Wire Wire Line
-	4550 6750 4550 6850
-Wire Wire Line
-	4550 6850 4650 6850
-Text Notes 5100 7250 0    50   ~ 0
-Addr: 0x69\n
-Wire Wire Line
 	4650 3350 4550 3350

Commit message: update
Parts:
- added TP6: TP_SDA, TestPoint:TestPoint_Pad_1.0x1.0mm, symbol Connector:TestPoint_Probe
- added TP7: TP_SCL, TestPoint:TestPoint_Pad_1.0x1.0mm, symbol Connector:TestPoint_Probe
- C30, C31, C32, C33, C34: footprint (none) -> Capacitor_SMD:C_0603_1608Metric_Pad1.05x0.95mm_HandSolder
- R4, R5: footprint (none) -> Resistor_SMD:R_0603_1608Metric_Pad1.05x0.95mm_HandSolder
Connections:
- net SCL: now also TP7.1
- net SDA: now also TP6.1
Changed lines of the file:
@@
 Text HLabel 900  1350 0    50   Input ~ 0
 SCL
-Text Label 1350 1250 0    50   ~ 0
+Text Label 1800 1250 0    50   ~ 0
 SDA
-Text Label 1350 1350 0    50   ~ 0
+Text Label 1800 1350 0    50   ~ 0
 SCL
 $Comp
@@
 F 0 "R4" H 950 1100 50  0000 L CNN
 F 1 "10k" H 900 1000 50  0000 L CNN
-F 2 "" H 1100 1050 50  0001 C CNN
+F 2 "Resistor_SMD:R_0603_1608Metric_Pad1.05x0.95mm_HandSolder" H 1100 1050 50  0001 C CNN
 F 3 "~" H 1100 1050 50  0001 C CNN
 	1    1100 1050
@@
 F 0 "R5" H 1259 1096 50  0000 L CNN
 F 1 "10k" H 1259 1005 50  0000 L CNN
-F 2 "" H 1200 1050 50  0001 C CNN
+F 2 "Resistor_SMD:R_0603_1608Metric_Pad1.05x0.95mm_HandSolder" H 1200 1050 50  0001 C CNN
 F 3 "~" H 1200 1050 50  0001 C CNN
 	1    1200 1050
@@
 F 0 "C33" H 6092 5446 50  0000 L CNN
 F 1 "0.1uF" H 6092 5355 50  0000 L CNN
-F 2 "" H 6000 5400 50  0001 C CNN
+F 2 "Capacitor_SMD:C_0603_1608Metric_Pad1.05x0.95mm_HandSolder" H 6000 5400 50  0001 C CNN
 F 3 "~" H 6000 5400 50  0001 C CNN
 	1    6000 5400
@@
 F 0 "C30" V 4821 1950 50  0000 C CNN
 F 1 "0.1uF" V 4912 1950 50  0000 C CNN
-F 2 "" H 5050 1950 50  0001 C CNN
+F 2 "Capacitor_SMD:C_0603_1608Metric_Pad1.05x0.95mm_HandSolder" H 5050 1950 50  0001 C CNN
 F 3 "~" H 5050 1950 50  0001 C CNN
 	1    5050 1950
@@
 F 0 "C34" V 5871 3350 50  0000 C CNN
 F 1 "0.1uF" V 5962 3350 50  0000 C CNN
-F 2 "" H 6100 3350 50  0001 C CNN
+F 2 "Capacitor_SMD:C_0603_1608Metric_Pad1.05x0.95mm_HandSolder" H 6100 3350 50  0001 C CNN
 F 3 "~" H 6100 3350 50  0001 C CNN
 	1    6100 3350
@@
 F 0 "C32" V 5250 1950 50  0000 C CNN
 F 1 "6.8nF" V 5350 1950 50  0000 C CNN
-F 2 "" H 5450 1950 50  0001 C CNN
+F 2 "Capacitor_SMD:C_0603_1608Metric_Pad1.05x0.95mm_HandSolder" H 5450 1950 50  0001 C CNN
 F 3 "~" H 5450 1950 50  0001 C CNN
 	1    5450 1950
@@
 F 0 "C31" V 5221 1600 50  0000 C CNN
 F 1 "120nF" V 5312 1600 50  0000 C CNN
-F 2 "" H 5450 1600 50  0001 C CNN
+F 2 "Capacitor_SMD:C_0603_1608Metric_Pad1.05x0.95mm_HandSolder" H 5450 1600 50  0001 C CNN
 F 3 "~" H 5450 1600 50  0001 C CNN
 	1    5450 1600
@@
 Text Notes 4700 5950 0    50   ~ 0
 Addr: 0x21\n
+$Comp
+L Connector:TestPoint_Probe TP?
+U 1 1 5E845BF0
+P 1350 1350
+AR Path="/5E845BF0" Ref="TP?"  Part="1"
+AR Path="/5E201923/5E845BF0" Ref="TP7"  Part="1"
+F 0 "TP7" H 1503 1451 50  0000 L CNN
+F 1 "TP_SCL" H 1503 1360 50  0000 L CNN
+F 2 "TestPoint:TestPoint_Pad_1.0x1.0mm" H 1550 1350 50  0001 C CNN
+F 3 "~" H 1550 1350 50  0001 C CNN
+	1    1350 1350
+	1    0    0    -1
+$EndComp
+$Comp
+L Connector:TestPoint_Probe TP?
+U 1 1 5E845BF6
+P 1350 1250
+AR Path="/5E845BF6" Ref="TP?"  Part="1"
+AR Path="/5E201923/5E845BF6" Ref="TP6"  Part="1"
+F 0 "TP6" H 1503 1351 50  0000 L CNN
+F 1 "TP_SDA" H 1503 1260 50  0000 L CNN
+F 2 "TestPoint:TestPoint_Pad_1.0x1.0mm" H 1550 1250 50  0001 C CNN
+F 3 "~" H 1550 1250 50  0001 C CNN
+	1    1350 1250
+	1    0    0    -1
+$EndComp
+Wire Wire Line
+	1350 1250 1800 1250
+Connection ~ 1350 1250
+Wire Wire Line
+	1350 1350 1800 1350
+Connection ~ 1350 1350
 $EndSCHEMATC

Commit message: first PCB
Connections:
- net SCL: now also U10.5 (SCL), U9.19 (COM1)
- net SDA: now also U10.8 (SDA), U9.20 (COM0)
Changed lines of the file:
@@
 Text Notes 6300 6050 0    50   ~ 0
 Can be connected to GND\n through different resistors\n for different addresses
-Text Notes 4150 3050 0    50   ~ 0
+Text Notes 3950 3050 0    50   ~ 0
 SDA
-Text Notes 4150 3150 0    50   ~ 0
+Text Notes 3800 3150 0    50   ~ 0
 SCL\n
 Text Notes 3800 3350 0    50   ~ 0
@@
 	1350 1350 1800 1350
 Connection ~ 1350 1350
+Text Label 4250 3050 2    50   ~ 0
+SDA
+Text Label 4150 3150 2    50   ~ 0
+SCL
 $EndSCHEMATC
