File: hardware/PCBs/Ragnarok_dev/Ragnarok_dev.kicad_pcb (KiCad board)
At the start: 2 copper layers, 3 parts, among them U1 BMP388, U2 FT232RL, U3 STM32F427VITx

Commit message: update
Parts:
- moved U2 68.1 mm to (78.7, 95.2)
- moved U3 56.4 mm to (102.9, 94.0)
- moved U1 44.4 mm to (119.4, 85.1)
Other:
- board outline added: 80 x 60 mm
Changed lines of the file:
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@@
-(kicad_pcb (version 20171130) (host pcbnew "(5.1.5-0-10_14)")
+(kicad_pcb (version 20171130) (host pcbnew "(5.1.5)-3")
   (general
     (thickness 1.6)
-    (drawings 0)
+    (drawings 4)
     (tracks 0)
     (zones 0)
@@
     (solder_mask_min_width 0.25)
     (aux_axis_origin 0 0)
-    (visible_elements FFFFFF7F)
+    (visible_elements 7FFFFFFF)
     (pcbplotparams
       (layerselection 0x010fc_ffffffff)
@@
   )
   (module BMP-388:PQFN50P200X200X80-10N (layer F.Cu)
-    (at 106.910001 42.495001)
+    (at 119.38 85.09)
     (fp_text reference U1 (at -0.284383 -1.605376) (layer F.SilkS)
       (effects (font (size 0.320434 0.320434) (thickness 0.015)))
@@
   )
   (module Package_SO:SSOP-28_5.3x10.2mm_P0.65mm (layer F.Cu)
-    (at 109.985001 34.735001)
+    (at 78.74 95.25)
     (descr "28-Lead Plastic Shrink Small Outline (SS)-5.30 mm Body [SSOP] (see Microchip Packaging Specification 00000049BS.pdf)")
     (tags "SSOP 0.65")
@@
   )
   (module Package_QFP:LQFP-100_14x14mm_P0.5mm (layer F.Cu)
-    (at 95.285001 38.135001)
+    (at 102.87 93.98)
     (descr "LQFP100: plastic low profile quad flat package; 100 leads; body 14 x 14 x 1.4 mm (see NXP sot407-1_po.pdf and sot407-1_fr.pdf)")
     (tags "QFP 0.5")
@@
     )
   )
+  (gr_line (start 62.85 124.44) (end 142.85 124.44) (layer Edge.Cuts) (width 0.12))
+  (gr_line (start 62.85 64.44) (end 62.85 124.44) (layer Edge.Cuts) (width 0.12))
+  (gr_line (start 62.85 64.44) (end 142.85 64.44) (layer Edge.Cuts) (width 0.12))
+  (gr_line (start 142.85 64.44) (end 142.85 124.44) (layer Edge.Cuts) (width 0.12))
 )

Commit message: finish schematic
Parts:
- added BT1: Battery, Connector_JST:JST_GH_SM02B-GHS-TB_1x02-1MP_P1.25mm_Horizontal, F.Cu at (164.7, 143.8)
- added C1: 0.1uF, Capacitor_SMD:C_0603_1608Metric_Pad1.05x0.95mm_HandSolder, F.Cu at (192.2, 135.3)
- added C10: 0.1uF, Capacitor_SMD:C_0603_1608Metric_Pad1.05x0.95mm_HandSolder, F.Cu at (186.0, 142.5)
- added C11: 0.1uF, Capacitor_SMD:C_0603_1608Metric_Pad1.05x0.95mm_HandSolder, F.Cu at (190.4, 142.5)
- added C12: 4.7uF, Capacitor_SMD:C_0603_1608Metric_Pad1.05x0.95mm_HandSolder, F.Cu at (182.4, 150.2)
- added C13: 0.1uF, Capacitor_SMD:C_0603_1608Metric_Pad1.05x0.95mm_HandSolder, F.Cu at (133.2, 195.6)
- added C14: 10nF, Capacitor_SMD:C_0603_1608Metric_Pad1.05x0.95mm_HandSolder, F.Cu at (151.2, 179.0)
- added C15: 10nF, Capacitor_SMD:C_0603_1608Metric_Pad1.05x0.95mm_HandSolder, F.Cu at (146.4, 183.9)
- added C16: 10nF, Capacitor_SMD:C_0603_1608Metric_Pad1.05x0.95mm_HandSolder, F.Cu at (142.0, 186.4)
- added C17: 10uF, Capacitor_SMD:C_0603_1608Metric_Pad1.05x0.95mm_HandSolder, F.Cu at (188.3, 145.0)
- added C18: 3.3nF, Capacitor_SMD:C_0603_1608Metric_Pad1.05x0.95mm_HandSolder, F.Cu at (192.6, 145.0)
- added C19: 22uF, Capacitor_SMD:C_0603_1608Metric_Pad1.05x0.95mm_HandSolder, F.Cu at (186.7, 150.2)
- added C2: 0.1uF, Capacitor_SMD:C_0603_1608Metric_Pad1.05x0.95mm_HandSolder, F.Cu at (187.9, 140.0)
- added C20: 0.1uF, Capacitor_SMD:C_0603_1608Metric_Pad1.05x0.95mm_HandSolder, F.Cu at (194.7, 140.4)
- added C21: 1uF, Capacitor_SMD:C_0603_1608Metric_Pad1.05x0.95mm_HandSolder, F.Cu at (186.7, 147.7)
- added C22: 0.1uF, Capacitor_SMD:C_0603_1608Metric_Pad1.05x0.95mm_HandSolder, F.Cu at (128.8, 196.5)
- added C23: 0.1uF, Capacitor_SMD:C_0603_1608Metric_Pad1.05x0.95mm_HandSolder, F.Cu at (124.2, 159.2)
- added C24: 1uF, Capacitor_SMD:C_0603_1608Metric_Pad1.05x0.95mm_HandSolder, F.Cu at (192.2, 137.9)
- added C25: 1uF, Capacitor_SMD:C_0603_1608Metric_Pad1.05x0.95mm_HandSolder, F.Cu at (183.9, 145.1)
- added C27: 0.1uF, Capacitor_SMD:C_0603_1608Metric_Pad1.05x0.95mm_HandSolder, F.Cu at (162.8, 163.7)
- added C28: 47pF, Capacitor_SMD:C_0603_1608Metric_Pad1.05x0.95mm_HandSolder, F.Cu at (170.1, 156.5)
- added C29: 0.1uF, Capacitor_SMD:C_0603_1608Metric_Pad1.05x0.95mm_HandSolder, F.Cu at (167.2, 163.7)
- added C3: 2.2uF, Capacitor_SMD:C_0603_1608Metric_Pad1.05x0.95mm_HandSolder, F.Cu at (183.5, 140.0)
- added C30: 0.1uF, Capacitor_SMD:C_0603_1608Metric_Pad1.05x0.95mm_HandSolder, F.Cu at (209.5, 139.9)
- added C31: 120nF, Capacitor_SMD:C_0603_1608Metric_Pad1.05x0.95mm_HandSolder, F.Cu at (213.1, 135.3)
- added C32: 6.8nF, Capacitor_SMD:C_0603_1608Metric_Pad1.05x0.95mm_HandSolder, F.Cu at (217.5, 132.8)
- added C33: 0.1uF, Capacitor_SMD:C_0603_1608Metric_Pad1.05x0.95mm_HandSolder, F.Cu at (209.5, 142.4)
- added C34: 0.1uF, Capacitor_SMD:C_0603_1608Metric_Pad1.05x0.95mm_HandSolder, F.Cu at (213.9, 137.9)
- added C35: 0.1uF, Capacitor_SMD:C_0603_1608Metric_Pad1.05x0.95mm_HandSolder, F.Cu at (136.0, 151.8)
- added C36: 0.1uF, Capacitor_SMD:C_0603_1608Metric_Pad1.05x0.95mm_HandSolder, F.Cu at (143.2, 150.2)
- added C4: 0.1uF, Capacitor_SMD:C_0603_1608Metric_Pad1.05x0.95mm_HandSolder, F.Cu at (181.7, 142.6)
- added C5: 1uF, Capacitor_SMD:C_0603_1608Metric_Pad1.05x0.95mm_HandSolder, F.Cu at (177.3, 142.6)
- added C6: 2.2uF, Capacitor_SMD:C_0603_1608Metric_Pad1.05x0.95mm_HandSolder, F.Cu at (187.9, 137.5)
- added C7: 0.1uF, Capacitor_SMD:C_0603_1608Metric_Pad1.05x0.95mm_HandSolder, F.Cu at (179.6, 145.1)
- added C8: 0.1uF, Capacitor_SMD:C_0603_1608Metric_Pad1.05x0.95mm_HandSolder, F.Cu at (193.9, 132.8)
- added C9: 0.1uF, Capacitor_SMD:C_0603_1608Metric_Pad1.05x0.95mm_HandSolder, F.Cu at (178.0, 148.4)
- added D1: 3V3, LED_SMD:LED_0603_1608Metric_Pad1.05x0.95mm_HandSolder, F.Cu at (131.7, 193.0)
- added D10: USB_PROTECTION, Diode_SMD:D_0603_1608Metric_Pad1.05x0.95mm_HandSolder, F.Cu at (170.9, 146.0)
- added D2: RX, LED_SMD:LED_0603_1608Metric_Pad1.05x0.95mm_HandSolder, F.Cu at (146.8, 178.0)
- added D3: TX, LED_SMD:LED_0603_1608Metric_Pad1.05x0.95mm_HandSolder, F.Cu at (131.7, 190.4)
- added D4: 5V, LED_SMD:LED_0603_1608Metric_Pad1.05x0.95mm_HandSolder, F.Cu at (124.5, 196.5)
- added D5: 6V, LED_SMD:LED_0603_1608Metric_Pad1.05x0.95mm_HandSolder, F.Cu at (137.7, 184.0)
- added D6: status, LED_SMD:LED_0603_1608Metric_Pad1.05x0.95mm_HandSolder, F.Cu at (120.1, 199.1)
- added D7: IR, Connector_JST:JST_GH_SM02B-GHS-TB_1x02-1MP_P1.25mm_Horizontal, F.Cu at (142.6, 173.0)
- added D8: D_Small, Diode_SMD:D_0603_1608Metric_Pad1.05x0.95mm_HandSolder, F.Cu at (120.1, 196.5)
- added D9: USB_PROTECTION, Diode_SMD:D_0603_1608Metric_Pad1.05x0.95mm_HandSolder, F.Cu at (169.3, 148.9)
- added FB1: FB?, Inductor_SMD:L_0603_1608Metric_Pad1.05x0.95mm_HandSolder, F.Cu at (178.0, 150.9)
- added FB2: FB, Inductor_SMD:L_0603_1608Metric_Pad1.05x0.95mm_HandSolder, F.Cu at (137.5, 197.9)
- added H1: MountingHole, MountingHole:MountingHole_2.2mm_M2, F.Cu at (141.6, 179.7)
- added H2: MountingHole, MountingHole:MountingHole_2.2mm_M2, F.Cu at (132.5, 180.2)
- added H3: MountingHole, MountingHole:MountingHole_2.2mm_M2, F.Cu at (132.5, 186.2)
- added H4: MountingHole, MountingHole:MountingHole_2.2mm_M2, F.Cu at (149.6, 172.2)
- added J1: USB_B_Micro, Connector_USB:USB_Micro-B_Amphenol_10103594-0001LF_Horizontal, F.Cu at (134.0, 173.1)
- added J2: BOARD_CONN, Connector_PinHeader_1.27mm:PinHeader_1x12_P1.27mm_Vertical_SMD_Pin1Left, F.Cu at (106.1, 177.9)
- added J3: BREAK_CONN, Connector_PinHeader_1.27mm:PinHeader_1x12_P1.27mm_Vertical_SMD_Pin1Right, F.Cu at (114.1, 177.9)
- added J4: JTAG, Connector_PinSocket_2.00mm:PinSocket_2x10_P2.00mm_Vertical, F.Cu at (100.0, 171.3)
- added J5: SPS30, Connector_JST:JST_GH_SM05B-GHS-TB_1x05-1MP_P1.25mm_Horizontal, F.Cu at (127.9, 154.3)
- added L1: 2.2uH, Inductor_SMD:L_0603_1608Metric_Pad1.05x0.95mm_HandSolder, F.Cu at (175.2, 145.9)
- added LS1: Buzzer, cmt-buzzer:CUI_CMT-8540S-SMT, F.Cu at (123.7, 174.8)
- added M1: Motor_DC, Connector_JST:JST_GH_SM02B-GHS-TB_1x02-1MP_P1.25mm_Horizontal, F.Cu at (125.5, 191.5)
- added M2: Motor_Servo, Connector_JST:JST_GH_SM03B-GHS-TB_1x03-1MP_P1.25mm_Horizontal, F.Cu at (170.3, 180.4)
- added M3: Motor_Servo, Connector_JST:JST_GH_SM03B-GHS-TB_1x03-1MP_P1.25mm_Horizontal, F.Cu at (170.3, 173.0)
- added M4: Motor_Servo, Connector_JST:JST_GH_SM03B-GHS-TB_1x03-1MP_P1.25mm_Horizontal, F.Cu at (161.1, 180.4)
- added M5: Motor_Servo, Connector_JST:JST_GH_SM03B-GHS-TB_1x03-1MP_P1.25mm_Horizontal, F.Cu at (161.1, 173.0)
- added M6: Motor_Servo, Connector_JST:JST_GH_SM03B-GHS-TB_1x03-1MP_P1.25mm_Horizontal, F.Cu at (179.6, 173.0)
- added Q1: NFET, Package_TO_SOT_SMD:SOT-23_Handsoldering, F.Cu at (105.3, 188.9)
- added Q2: NFET, Package_TO_SOT_SMD:SOT-23_Handsoldering, F.Cu at (114.7, 197.2)
- added Q3: Q_NMOS_GSD, Package_TO_SOT_SMD:SOT-23_Handsoldering, F.Cu at (171.9, 142.4)
- added Q4: Q_PMOS_GSD, Package_TO_SOT_SMD:SOT-23_Handsoldering, F.Cu at (163.9, 149.8)
- added Q5: Q_PMOS_GSD, Package_TO_SOT_SMD:SOT-23_Handsoldering, F.Cu at (179.3, 133.9)
- added R1: 270, Resistor_SMD:R_0603_1608Metric_Pad1.05x0.95mm_HandSolder, F.Cu at (142.0, 183.9)
- added R10: 300, Resistor_SMD:R_0603_1608Metric_Pad1.05x0.95mm_HandSolder, F.Cu at (136.1, 192.9)
- added R11: 400, Resistor_SMD:R_0603_1608Metric_Pad1.05x0.95mm_HandSolder, F.Cu at (128.8, 199.0)
- added R12: 300, Resistor_SMD:R_0603_1608Metric_Pad1.05x0.95mm_HandSolder, F.Cu at (140.4, 189.0)
- added R13: 4.7k, Resistor_SMD:R_0603_1608Metric_Pad1.05x0.95mm_HandSolder, F.Cu at (133.2, 198.1)
- added R14: 300, Resistor_SMD:R_0603_1608Metric_Pad1.05x0.95mm_HandSolder, F.Cu at (140.4, 191.5)
- added R15: 10k, Resistor_SMD:R_0603_1608Metric_Pad1.05x0.95mm_HandSolder, F.Cu at (137.5, 195.4)
- added R16: 10k, Resistor_SMD:R_0603_1608Metric_Pad1.05x0.95mm_HandSolder, F.Cu at (151.1, 181.5)
- added R17: 10k, Resistor_SMD:R_0603_1608Metric_Pad1.05x0.95mm_HandSolder, F.Cu at (146.4, 186.4)
- added R18: 10k, Resistor_SMD:R_0603_1608Metric_Pad1.05x0.95mm_HandSolder, F.Cu at (144.8, 188.9)
- added R19: 10k, Resistor_SMD:R_0603_1608Metric_Pad1.05x0.95mm_HandSolder, F.Cu at (173.7, 148.5)
- added R2: 270, Resistor_SMD:R_0603_1608Metric_Pad1.05x0.95mm_HandSolder, F.Cu at (137.6, 186.5)
- added R20: 10k, Resistor_SMD:R_0603_1608Metric_Pad1.05x0.95mm_HandSolder, F.Cu at (189.6, 132.8)
- added R21: 10k, Resistor_SMD:R_0603_1608Metric_Pad1.05x0.95mm_HandSolder, F.Cu at (183.5, 137.5)
- added R3: 100k, Resistor_SMD:R_0603_1608Metric_Pad1.05x0.95mm_HandSolder, F.Cu at (182.4, 147.7)
- added R4: 10k, Resistor_SMD:R_0603_1608Metric_Pad1.05x0.95mm_HandSolder, F.Cu at (217.5, 135.3)
- added R5: 10k, Resistor_SMD:R_0603_1608Metric_Pad1.05x0.95mm_HandSolder, F.Cu at (213.1, 132.8)
- added R6: 31.6k, Resistor_SMD:R_0603_1608Metric_Pad1.05x0.95mm_HandSolder, F.Cu at (124.5, 199.1)
- added R7: 12k, Resistor_SMD:R_0603_1608Metric_Pad1.05x0.95mm_HandSolder, F.Cu at (136.1, 190.4)
- added R8: 10k, Resistor_SMD:R_0603_1608Metric_Pad1.05x0.95mm_HandSolder, F.Cu at (146.8, 180.6)
- added R9: 300, Resistor_SMD:R_0603_1608Metric_Pad1.05x0.95mm_HandSolder, F.Cu at (151.2, 176.5)
- added SW1: Programming, CS12 Switch:CS12ANW03, F.Cu at (103.7, 195.7)
- added SW2: SW_Push, Button_Switch_SMD:SW_SPST_B3SL-1022P, F.Cu at (116.5, 190.8)
- added SW3: Power, CS12 Switch:CS12ANW03, F.Cu at (168.4, 136.0)
- added TH1: 10k@25, Connector_JST:JST_GH_SM02B-GHS-TB_1x02-1MP_P1.25mm_Horizontal, F.Cu at (125.5, 184.0)
- added TP1: TP_USBTX, TestPoint:TestPoint_Pad_1.0x1.0mm, F.Cu at (119.7, 181.8)
- added TP2: TP_USBRX, TestPoint:TestPoint_Pad_1.0x1.0mm, F.Cu at (119.7, 184.9)
- added TP3: TP_SCLK, TestPoint:TestPoint_Pad_1.0x1.0mm, F.Cu at (173.4, 159.8)
- added TP4: TP_MOSI, TestPoint:TestPoint_Pad_1.0x1.0mm, F.Cu at (173.8, 156.7)
- added TP5: TP_MISO, TestPoint:TestPoint_Pad_1.0x1.0mm, F.Cu at (176.8, 156.7)
- added TP6: TP_SDA, TestPoint:TestPoint_Pad_1.0x1.0mm, F.Cu at (221.2, 133.1)
- added TP7: TP_SCL, TestPoint:TestPoint_Pad_1.0x1.0mm, F.Cu at (213.2, 140.6)
- added U1: ublox_SAM-M8Q, RF_Module:ublox_SAM-M8Q_HandSolder, F.Cu at (131.5, 141.1)
- added U10: SDP32, SDP32-125PA-TR-250PCS:XDCR_SDP32-125PA-TR-250PCS, F.Cu at (206.0, 135.1)
- added U11: Openlog, Connector_PinHeader_2.54mm:PinHeader_1x06_P2.54mm_Vertical, F.Cu at (143.3, 133.9)
- added U12: MiniSpy, Connector_JST:JST_GH_SM03B-GHS-TB_1x03-1MP_P1.25mm_Horizontal, F.Cu at (179.6, 180.4)
- added U2: XBP9B-DMST-002, xbee:DIP2200W51P200L3294H279Q20P, F.Cu at (109.0, 148.9)
- added U5: TPS62142, Package_DFN_QFN:QFN-16-1EP_3x3mm_P0.5mm_EP1.8x1.8mm, F.Cu at (178.7, 138.8)
- added U6: RT9069-50GB, Package_TO_SOT_SMD:SOT-23-5, F.Cu at (185.0, 133.9)
- added U7: AB0815, Package_DFN_QFN:QFN-16-1EP_5x5mm_P0.8mm_EP2.7x2.7mm, F.Cu at (164.3, 158.8)
- added U8: BMP388, BMP-388:PQFN50P200X200X80-10N, F.Cu at (170.1, 159.5)
- added U9: BNO055, Package_LGA:LGA-28_5.2x3.8mm_P0.5mm, F.Cu at (203.9, 141.4)
- moved U1 68.9 mm to (113.0, 153.7)
- renumbered U2 to U3, U3 to U4
Connections:
- net Net-(U3-Pad78) renamed /UART/XB_TX
- net Net-(U3-Pad79) renamed /UART/XB_RX
- net Net-(U3-Pad86) renamed /GPS_TX
- net Net-(U3-Pad87) renamed /GPS_RX
- U3 pad 1: Net-(U2-Pad1) -> /USB_RX
- U3 pad 18: Net-(U2-Pad18) -> GND
- U3 pad 20: Net-(U2-Pad20) -> Net-(C15-Pad1)
- U3 pad 21: Net-(U2-Pad21) -> GND
- U3 pad 25: Net-(U2-Pad25) -> GND
- U3 pad 4: Net-(U2-Pad4) -> Net-(C15-Pad1)
- U3 pad 5: Net-(U2-Pad5) -> /USB_TX
- U3 pad 7: Net-(U2-Pad7) -> GND
- U4 pad 10: Net-(U3-Pad10) (its old number) -> GND
- U4 pad 100: Net-(U3-Pad100) -> +3V3
- U4 pad 11: Net-(U3-Pad11) (its old number) -> +3V3
- U4 pad 19: Net-(U3-Pad19) (its old number) -> +3V3
- U4 pad 20: Net-(U3-Pad20) -> GND
- U4 pad 21: Net-(U3-Pad21) -> +3V3
- U4 pad 22: Net-(U3-Pad22) -> /Power Supply/MCU_AVDD
- U4 pad 24: Net-(U3-Pad24) -> /voltage_div
- U4 pad 25: Net-(U3-Pad25) -> /voltage_therm
- U4 pad 27: Net-(U3-Pad27) (its old number) -> GND
- U4 pad 28: Net-(U3-Pad28) (its old number) -> +3V3
- U4 pad 30: Net-(U3-Pad30) -> /SPI Sensors/SCLK
- U4 pad 31: Net-(U3-Pad31) -> /SPI Sensors/MISO
- U4 pad 32: Net-(U3-Pad32) -> /SPI Sensors/MOSI
- U4 pad 33: Net-(U3-Pad33) -> /BMP_CSB
- U4 pad 34: Net-(U3-Pad34) -> /ABO_CSB
- U4 pad 37: Net-(U3-Pad37) -> /IR_TRANSMIT
- U4 pad 47: Net-(U3-Pad47) -> /I2C Sensors/SCL
- U4 pad 48: Net-(U3-Pad48) -> /I2C Sensors/SDA
- U4 pad 49: Net-(U3-Pad49) -> +3V3
- U4 pad 50: Net-(U3-Pad50) -> +3V3
- U4 pad 64: Net-(U3-Pad64) -> /Servo5
- U4 pad 67: Net-(U3-Pad67) -> /Servo1
- U4 pad 68: Net-(U3-Pad68) -> /Servo2
- U4 pad 69: Net-(U3-Pad69) -> /Servo3
- U4 pad 7: Net-(U3-Pad7) -> /status_led
- U4 pad 70: Net-(U3-Pad70) -> /Servo4
- U4 pad 71: Net-(U3-Pad71) -> /Cam
- U4 pad 72: Net-(U3-Pad72) -> /TMS
- U4 pad 73: Net-(U3-Pad73) -> +3V3
- U4 pad 74: Net-(U3-Pad74) -> GND
- U4 pad 75: Net-(U3-Pad75) -> +3V3
- U4 pad 76: Net-(U3-Pad76) -> /TCK
- U4 pad 77: Net-(U3-Pad77) -> /JTDI
- U4 pad 80: Net-(U3-Pad80) -> /UART/LOG_TX
- U4 pad 83: Net-(U3-Pad83) -> /LOG_RX
- U4 pad 89: Net-(U3-Pad89) -> /JTDO
- U4 pad 90: Net-(U3-Pad90) -> /nTRST
- U4 pad 92: Net-(U3-Pad92) -> /USB_TX
- U4 pad 93: Net-(U3-Pad93) -> /USB_RX
- U4 pad 95: Net-(U3-Pad95) -> /speaker_driver
- U4 pad 96: Net-(U3-Pad96) -> /motor_driver
- U4 pad 97: Net-(U3-Pad97) -> /SPS_RX
- U4 pad 98: Net-(U3-Pad98) -> /SPS_TX
- U4 pad 99: Net-(U3-Pad99) -> GND

Commit message: begin layout
Parts:
- removed the U1 at (113.0, 153.7)
- added H5: MountingHole, MountingHole:MountingHole_2.2mm_M2, F.Cu at (151.1, 68.6)
- added H6: MountingHole, MountingHole:MountingHole_2.2mm_M2, F.Cu at (149.9, 120.7)
- added H7: MountingHole, MountingHole:MountingHole_2.2mm_M2, F.Cu at (221.0, 68.6)
- added H8: MountingHole, MountingHole:MountingHole_2.2mm_M2, F.Cu at (221.0, 119.4)
- R10, R11, R12, R9: moved to B.Cu
- moved C17 139.0 mm to (81.7, 55.9)
- moved C19 136.2 mm to (81.7, 63.5)
- moved C18 135.5 mm to (86.4, 61.0)
- moved H3 135.1 mm to (66.0, 68.6)
- moved R3 132.9 mm to (81.7, 61.0)
- moved L1 127.2 mm to (82.9, 58.4)
- moved R13 124.9 mm to (112.2, 74.9)
- moved SW2 124.2 mm to (115.2, 66.6)
- moved SW1 123.5 mm to (72.4, 76.2)
- moved C24 121.3 mm to (88.5, 74.9)
- moved C25 119.6 mm to (88.7, 72.8)
- moved U6 118.1 mm to (84.0, 72.7)
- moved U5 118.0 mm to (83.8, 68.6)
- moved BT1 117.9 mm to (74.9, 67.3), turned to 180 degrees
- moved R20 113.0 mm to (89.2, 80.8)
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Other:
- board size 80 x 60 mm -> 162.6 x 60 mm

Commit message: first PCB
Parts:
- C13, C14, C15, C16, C30, C31, C32, C33, C34, D10, FB2, LS1, Q1, Q3, Q4, Q5, R1, R13, R19, R2, R20, R21, TP1, TP2, U10, U3, U9: moved to B.Cu
- J2: footprint Connector_PinHeader_1.27mm:PinHeader_1x12_P1.27mm_Vertical_SMD_Pin1Left -> ragnarok_custom_libs:Board_Jumper
- J3: footprint Connector_PinHeader_1.27mm:PinHeader_1x12_P1.27mm_Vertical_SMD_Pin1Right -> ragnarok_custom_libs:Board_Jumper
- moved C22 104.2 mm to (107.7, 69.5), turned to 270 degrees
- moved R15 96.4 mm to (102.5, 77.7)
- moved R16 84.4 mm to (70.1, 102.7), turned to 270 degrees
- moved R18 80.6 mm to (67.3, 111.9), turned to 180 degrees
- moved R17 80.1 mm to (70.2, 108.7), turned to 270 degrees
- moved R6 74.1 mm to (96.1, 102.9)
- moved R7 69.7 mm to (96.1, 101.5)
- moved TP2 65.5 mm to (82.3, 99.6)
- moved R8 62.7 mm to (96.2, 104.3), turned to 180 degrees
- moved TP1 61.0 mm to (82.3, 101.2)
- moved H7 58.4 mm to (162.6, 68.6)
- moved H8 58.2 mm to (162.8, 121.5)
- moved U8 58.1 mm to (131.5, 80.2)
- moved M6 57.6 mm to (156.0, 68.5), turned to 180 degrees
- moved C29 57.5 mm to (128.9, 80.4), turned to 270 degrees
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Connections:
- J3 pad 1: /Breakout/+6 -> GND
- J3 pad 10: GND -> /Breakout/+5
- J3 pad 11: GND -> /Breakout/+6
- J3 pad 12: GND -> /Breakout/+6
- J3 pad 2: /Breakout/+6 -> GND
- J3 pad 3: /Breakout/+5 -> GND
- J3 pad 4: /Breakout/Servo1 -> /Breakout/Cam
- J3 pad 5: /Breakout/Servo2 -> /Breakout/Servo5
- J3 pad 6: /Breakout/Servo3 -> /Breakout/Servo4
- J3 pad 7: /Breakout/Servo4 -> /Breakout/Servo3
- J3 pad 8: /Breakout/Servo5 -> /Breakout/Servo2
- J3 pad 9: /Breakout/Cam -> /Breakout/Servo1
- U1 pad 13: /UART/RX_SAM -> /GPS_RX
- U1 pad 14: /UART/TX_SAM -> /GPS_TX
- U10 pad 5: Net-(U10-Pad5) -> /I2C Sensors/SCL
- U10 pad 8: Net-(U10-Pad8) -> /I2C Sensors/SDA
- U2 pad 2: /UART/XBEE_RX -> /UART/XB_RX
- U2 pad 3: /UART/XBEE_TX -> /UART/XB_TX
- U9 pad 19: Net-(U10-Pad5) -> /I2C Sensors/SCL
- U9 pad 20: Net-(U10-Pad8) -> /I2C Sensors/SDA
Routing:
- net GND: track 0.00 -> 398.8 mm, vias 0 -> 51
- net +3V3: track 0.00 -> 363.3 mm, vias 0 -> 11
- net +6V: track 0.00 -> 173.9 mm, vias 0 -> 10
- net +5V: track 0.00 -> 160.8 mm, vias 0 -> 3
- net /SPI Sensors/SCLK: track 0.00 -> 92.6 mm, vias 0 -> 5
- net /SPI Sensors/MISO: track 0.00 -> 88.7 mm, vias 0 -> 4
- net /SPI Sensors/MOSI: track 0.00 -> 85.0 mm, vias 0 -> 6
- net /BMP_CSB: track 0.00 -> 75.3 mm, vias 0 -> 4
- net /ABO_CSB: track 0.00 -> 64.6 mm, vias 0 -> 4
- net Net-(D9-Pad1): track 0.00 -> 61.2 mm, vias 0 -> 1
- net /TMS: track 0.00 -> 60.1 mm, vias 0 -> 3
- net /JTDI: track 0.00 -> 60.1 mm, vias 0 -> 3
- net /TCK: track 0.00 -> 59.7 mm, vias 0 -> 3
- net /Breakout/+6: track 0.00 -> 59.1 mm
- net /Breakout/Servo5: track 0.00 -> 58.5 mm
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- added copper zone on B.Cu, net GND
- added copper zone on F.Cu, net GND
Other:
- board size 162.6 x 60 mm -> 102.7 x 60 mm
- board text added: "OFF"
- board text added: "ON"
- board text added: "RUN"

Commit message: final changes
Parts:
- moved H6 2.35 mm to (148.4, 119.4)
- moved H1 2.21 mm to (137.8, 119.4)
- moved H2 2.18 mm to (67.8, 119.4)
- moved H8 2.12 mm to (162.5, 119.4)
- moved H4 2.04 mm to (137.8, 69.4)
- moved H3 2.00 mm to (67.8, 69.4)
- moved H7 0.86 mm to (162.5, 69.4)
- moved H5 0.86 mm to (148.4, 69.4)
Routing:
- net GND: track 398.8 -> 426.9 mm, vias 51 -> 54
Other:
- board text added: "Ragnarok Development March 2020"
